Commit message: Update the human model to be closer to kinect skeleton
- Rename multiple links to avoid confusion between joints and links
- Change base frame to base instead of hip
- Add one more DOF in the back via spine joint
- Change lengths of multiple segments

File: urdf/xacro/human_arm.urdf.xacro (robot description, xacro)
@@ -6,5 +6,5 @@
     <link name="${side}_shoulder_0"/>
     <link name="${side}_shoulder_1"/>
-    <link name="${side}_upper_arm">
+    <link name="${side}_shoulder">
       <visual>
         <origin xyz="${upper_arm_length/2} 0 0" rpy="0 ${PI_DIV_2} 0" />
@@ -15,5 +15,5 @@
     </link>
     <link name="${side}_elbow_0"/>
-    <link name="${side}_forearm">
+    <link name="${side}_elbow">
       <visual>
         <origin xyz="${forearm_length/2} 0 0" rpy="0 ${PI_DIV_2} 0" />
@@ -24,5 +24,5 @@
     </link>
     <link name="${side}_wrist_0"/>
-    <link name="${side}_hand">
+    <link name="${side}_wrist">
       <visual>
         <origin xyz="${hand_length/2} 0 0" rpy="0 0 0" />
@@ -32,9 +32,9 @@
       </visual>
     </link>
-    <link name="${side}_hand_tip"/>
+    <link name="${side}_hand"/>
     <!-- Joints -->
     <joint name="${side}_arm_mount" type="fixed">
-      <origin xyz="0 ${reflect*shoulder_offset_width} ${shoulder_offset_height}" rpy="0 0 ${reflect*PI_DIV_2}" />
-      <parent link="torso" />
+      <origin xyz="0 ${reflect*shoulder_offset_width} 0" rpy="0 0 ${reflect*PI_DIV_2}" />
+      <parent link="shoulder_center" />
       <child link="${side}_arm_mount" />
     </joint>
@@ -69,5 +69,5 @@
           <axis xyz="1 0 0" />
           <parent link="${side}_shoulder_1" />
-          <child link="${side}_upper_arm" />
+          <child link="${side}_shoulder" />
           <limit lower="${-PI_DIV_2}" upper="${PI_DIV_2}" effort="${max_effort}" velocity="${max_velocity}"  />
         </joint>
@@ -77,5 +77,5 @@
         <origin xyz="${upper_arm_length} 0 0" rpy="0 0 0" />
         <axis xyz="0 0 1" />
-        <parent link="left_upper_arm" />
+        <parent link="left_shoulder" />
         <child link="left_elbow_0" />
         <limit lower="${-PI}" upper="0.0" effort="${max_effort}" velocity="${max_velocity}"  />
@@ -85,5 +85,5 @@
         <axis xyz="1 0 0" />
         <parent link="left_elbow_0" />
-        <child link="left_forearm" />
+        <child link="left_elbow" />
         <limit lower="${-PI}" upper="0.0" effort="${max_effort}" velocity="${max_velocity}"  />
       </joint>
@@ -93,5 +93,5 @@
         <origin xyz="${upper_arm_length} 0 0" rpy="0 0 0" />
         <axis xyz="0 0 1" />
-        <parent link="right_upper_arm" />
+        <parent link="right_shoulder" />
         <child link="right_elbow_0" />
         <limit lower="0.0" upper="${PI}" effort="${max_effort}" velocity="${max_velocity}"  />
@@ -101,5 +101,5 @@
         <axis xyz="1 0 0" />
         <parent link="right_elbow_0" />
-        <child link="right_forearm" />
+        <child link="right_elbow" />
         <limit lower="0.0" upper="${PI}" effort="${max_effort}" velocity="${max_velocity}"  />
       </joint>
@@ -108,5 +108,5 @@
       <origin xyz="${forearm_length} 0 0" rpy="0 0 0" />
       <axis xyz="0 0 1" />
-      <parent link="${side}_forearm" />
+      <parent link="${side}_elbow" />
       <child link="${side}_wrist_0" />
       <limit lower="${-PI_DIV_4}" upper="${PI_DIV_4}" effort="${max_effort}" velocity="${max_velocity}"  />
@@ -116,11 +116,11 @@
       <axis xyz="0 1 0" />
       <parent link="${side}_wrist_0" />
-      <child link="${side}_hand" />
+      <child link="${side}_wrist" />
       <limit lower="${-PI_DIV_2}" upper="${PI_DIV_2}" effort="${max_effort}" velocity="${max_velocity}"  />
     </joint>
     <joint name="${side}_hand" type="fixed">
       <origin xyz="${hand_length} 0 0" rpy="0 0 0" />
-      <parent link="${side}_hand" />
-      <child link="${side}_hand_tip" />
+      <parent link="${side}_wrist" />
+      <child link="${side}_hand" />
     </joint>
 </xacro:macro>

File: urdf/xacro/human_body.urdf.xacro (robot description, xacro)
@@ -3,22 +3,40 @@
 <xacro:include filename="props_global.urdf.xacro" />
 <xacro:macro name="human_body">
-	<link name="hip"/>
-    <link name="waist">
+	<link name="base"/>
+    <link name="hip">
       <visual>
         <origin xyz="0 0 ${waist_length/2}" rpy="0 0 0" />
         <geometry>
-	        <!--<box size="0.4 0.2 ${waist_length}" />-->
-	        <cylinder radius="${waist_radius}" length="${waist_length}" />
+          <!--<box size="0.4 0.2 ${waist_length}" />-->
+          <cylinder radius="${waist_radius}" length="${waist_length}" />
         </geometry>
       </visual>
     </link>
-	<link name="spine_0"/>
-    <link name="spine_1"/>
-    <link name="torso">
+    <link name="waist_0"/>
+    <link name="waist_1"/>
+    <link name="waist">
+      <visual>
+        <origin xyz="0 0 ${spine_down_length/2}" rpy="0 0 0" />
+        <geometry>
+          <!--<box size="0.4 0.2 ${torso_length}" />-->
+          <cylinder radius="${spine_radius}" length="${spine_down_length}" />
+        </geometry>
+      </visual>
+    </link>
+    <link name="spine">
+      <visual>
+        <origin xyz="0 0 ${spine_up_length/2}" rpy="0 0 0" />
+        <geometry>
+	        <!--<box size="0.4 0.2 ${torso_length}" />-->
+	        <cylinder radius="${spine_radius}" length="${spine_up_length}" />
+        </geometry>
+      </visual>
+    </link>
+    <link name="shoulder_center">
       <visual>
         <origin xyz="0 0 ${torso_length/2}" rpy="0 0 0" />
         <geometry>
-	        <!--<box size="0.4 0.2 ${torso_length}" />-->
-	        <cylinder radius="${torso_radius}" length="${torso_length}" />
+          <!--<box size="0.4 0.2 ${torso_length}" />-->
+          <cylinder radius="${torso_radius}" length="${torso_length}" />
         </geometry>
       </visual>
@@ -26,7 +44,16 @@
     <link name="neck_0"/>
     <link name="neck_1"/>
+    <link name="neck">
+      <visual>
+        <origin xyz="0 0 ${neck_length/2}" rpy="0 0 0" />
+        <geometry>
+          <!--<box size="0.4 0.2 ${torso_length}" />-->
+          <cylinder radius="${neck_radius}" length="${neck_length}" />
+        </geometry>
+      </visual>
+    </link>
     <link name="head">
       <visual>
-        <origin xyz="0 0 ${neck_length}" rpy="0 0 0" />
+        <origin xyz="0 0 0" rpy="0 0 0" />
         <geometry>
 	        <sphere radius="${head_radius}" />
@@ -34,31 +61,42 @@
       </visual>
     </link>
-    <link name="head_tip"/>
     <joint name="hip" type="fixed">
       <origin xyz="0 0 0" rpy="0 0 0" />
-      <parent link="hip" />
-      <child link="waist" />
+      <parent link="base" />
+      <child link="hip" />
     </joint>
     <!-- SPINE : spherical -->
-    <joint name="spine_0" type="revolute">
+    <joint name="waist_0" type="revolute">
       <origin xyz="0 0 ${waist_length}" rpy="0 0 0" />
       <axis xyz="1 0 0" />
-      <parent link="waist" />
-      <child link="spine_0" />
+      <parent link="hip" />
+      <child link="waist_0" />
       <limit lower="${-PI_DIV_2}" upper="${PI_DIV_2}" effort="${max_effort}" velocity="${max_velocity}" />
     </joint>
-    <joint name="spine_1" type="revolute">
+    <joint name="waist_1" type="revolute">
       <origin xyz="0 0 0" rpy="0 0 0" />
       <axis xyz="0 1 0" />
-      <parent link="spine_0" />
-      <child link="spine_1" />
+      <parent link="waist_0" />
+      <child link="waist_1" />
       <limit lower="${-PI_DIV_2}" upper="${PI_DIV_2}" effort="${max_effort}" velocity="${max_velocity}" />
     </joint>
-    <joint name="spine_2" type="revolute">
+    <joint name="waist_2" type="revolute">
       <origin xyz="0 0 0" rpy="0 0 0" />
       <axis xyz="0 0 1" />
-      <parent link="spine_1" />
-      <child link="torso" />
+      <parent link="waist_1" />
+      <child link="waist" />
       <limit lower="${-PI_DIV_2}" upper="${PI_DIV_2}" effort="${max_effort}" velocity="${max_velocity}" />
+    </joint>
+    <joint name="spine" type="revolute">
+      <origin xyz="0 0 ${spine_down_length}" rpy="0 0 0" />
+      <axis xyz="0 1 0" />
+      <parent link="waist" />
+      <child link="spine" />
+      <limit lower="${-PI_DIV_2}" upper="${PI_DIV_2}" effort="${max_effort}" velocity="${max_velocity}" />
+    </joint>
+    <joint name="shoulder_center" type="fixed">
+      <origin xyz="0 0 ${spine_up_length}" rpy="0 0 0" />
+      <parent link="spine" />
+      <child link="shoulder_center" />
     </joint>
     <!-- NECK : spherical -->
@@ -66,5 +104,5 @@
           <origin xyz="0 0 ${torso_length}" rpy="0 0 0" />
           <axis xyz="1 0 0" />
-          <parent link="torso" />
+          <parent link="shoulder_center" />
           <child link="neck_0" />
           <limit lower="${-PI_DIV_2}" upper="${PI_DIV_2}" effort="${max_effort}" velocity="${max_velocity}"  />
@@ -81,5 +119,5 @@
           <axis xyz="0 0 1" />
           <parent link="neck_1" />
-          <child link="head" />
+          <child link="neck" />
           <limit lower="${-PI_DIV_2}" upper="${PI_DIV_2}" effort="${max_effort}" velocity="${max_velocity}" />
         </joint>
@@ -87,6 +125,6 @@
     <joint name="head" type="fixed">
       <origin xyz="0 0 ${neck_length}" rpy="0 0 0" />
-      <parent link="head" />
-      <child link="head_tip" />
+      <parent link="neck" />
+      <child link="head" />
     </joint>
 </xacro:macro>

File: urdf/xacro/human_leg.urdf.xacro (robot description, xacro)
@@ -6,5 +6,5 @@
     <link name="${side}_hip_0"/>
     <link name="${side}_hip_1"/>
-    <link name="${side}_thigh">
+    <link name="${side}_hip">
       <visual>
         <origin xyz="${thigh_length/2} 0 0" rpy="0 ${PI_DIV_2} 0" />
@@ -14,5 +14,5 @@
       </visual>
     </link>
-    <link name="${side}_shin">
+    <link name="${side}_knee">
       <visual>
         <origin xyz="${shin_length/2} 0 0" rpy="0 ${PI_DIV_2} 0" />
@@ -22,6 +22,6 @@
       </visual>
     </link>
-    <link name="${side}_ankle"/>
-    <link name="${side}_foot">
+    <link name="${side}_ankle_0"/>
+    <link name="${side}_ankle">
       <visual>
         <origin xyz="${foot_length/2} 0 0" rpy="0 0 0" />
@@ -31,9 +31,9 @@
       </visual>
     </link>
-    <link name="${side}_foot_tip"/>
+    <link name="${side}_foot"/>
     <!-- Joints -->
     <joint name="${side}_hip_leg_mount" type="fixed">
-      <origin xyz="0 ${reflect*hip_offset_width} ${hip_offset_height}" rpy="0 ${PI_DIV_2} 0" />
-      <parent link="hip" />
+      <origin xyz="0 ${reflect*hip_offset_width} 0" rpy="0 ${PI_DIV_2} 0" />
+      <parent link="base" />
       <child link="${side}_leg_mount" />
     </joint>
@@ -57,5 +57,5 @@
           <axis xyz="1 0 0" />
           <parent link="${side}_hip_1" />
-          <child link="${side}_thigh" />
+          <child link="${side}_hip" />
           <limit lower="${-PI_DIV_2}" upper="${PI_DIV_2}" effort="${max_effort}" velocity="${max_velocity}"  />
         </joint>
@@ -64,6 +64,6 @@
       <origin xyz="${thigh_length} 0 0" rpy="${PI_DIV_2} 0 0" />
       <axis xyz="0 0 1" />
-      <parent link="${side}_thigh" />
-      <child link="${side}_shin" />
+      <parent link="${side}_hip" />
+      <child link="${side}_knee" />
       <limit lower="${-PI}" upper="0.1" effort="${max_effort}" velocity="${max_velocity}"  />
     </joint>
@@ -72,6 +72,6 @@
           <origin xyz="${shin_length} 0 0" rpy="${-PI_DIV_2} 0 ${PI_DIV_2}" />
           <axis xyz="0 0 1" />
-          <parent link="${side}_shin" />
-          <child link="${side}_ankle" />
+          <parent link="${side}_knee" />
+          <child link="${side}_ankle_0" />
           <limit lower="${-PI_DIV_2}" upper="${PI_DIV_2}" effort="${max_effort}" velocity="${max_velocity}"  />
         </joint>
@@ -79,6 +79,6 @@
           <origin xyz="0 0 0" rpy="0 0 0" />
           <axis xyz="0 1 0" />
-          <parent link="${side}_ankle" />
-          <child link="${side}_foot" />
+          <parent link="${side}_ankle_0" />
+          <child link="${side}_ankle" />
           <limit lower="${-PI_DIV_2}" upper="${PI_DIV_2}" effort="${max_effort}" velocity="${max_velocity}" />
         </joint>
@@ -86,6 +86,6 @@
     <joint name="${side}_foot" type="fixed">
       <origin xyz="${foot_length} 0 0" rpy="0 0 0" />
-      <parent link="${side}_foot" />
-      <child link="${side}_foot_tip" />
+      <parent link="${side}_ankle" />
+      <child link="${side}_foot" />
     </joint>
 </xacro:macro>

File: urdf/xacro/props_global.urdf.xacro (robot description, xacro)
@@ -15,14 +15,16 @@
   <xacro:property name="torso_length" value="$(arg torso_length)" />
   <xacro:property name="torso_radius" value="$(arg torso_radius)" />
+  <xacro:property name="waist_length" value="$(arg waist_length)" />
   <xacro:property name="waist_radius" value="$(arg waist_radius)" />
-  <xacro:property name="waist_length" value="$(arg waist_length)" />
+  <xacro:property name="spine_down_length" value="$(arg spine_down_length)" />
+  <xacro:property name="spine_up_length" value="$(arg spine_up_length)" />
+  <xacro:property name="spine_radius" value="$(arg spine_radius)" />
   <xacro:property name="neck_length" value="$(arg neck_length)" />
+  <xacro:property name="neck_radius" value="$(arg neck_radius)" />
   <xacro:property name="thigh_length" value="$(arg thigh_length)" />
   <xacro:property name="shin_length" value="$(arg shin_length)" />
   <xacro:property name="foot_length" value="$(arg foot_length)" />
   <xacro:property name="shoulder_offset_width" value="$(arg shoulder_offset_width)" />
-  <xacro:property name="shoulder_offset_height" value="$(arg shoulder_offset_height)" />
   <xacro:property name="hip_offset_width" value="$(arg hip_offset_width)" />
-  <xacro:property name="hip_offset_height" value="$(arg hip_offset_height)" />
   <xacro:property name="max_effort" value="1" />
   <xacro:property name="max_velocity" value="1" />
