Commit message: Replace /human prefix by human to avoid tf2 troubles

File: urdf/xacro/props_global.urdf.xacro (robot description, xacro)
@@ -1,5 +1,5 @@
 <?xml version="1.0"?>
 <robot xmlns:xacro="http://playerstage.sourceforge.net/gazebo/xmlschema/#interface" name="human_model" >
-  <xacro:property name="prefix" value="/human" />
+  <xacro:property name="prefix" value="human" />
   <xacro:property name="PI" value="3.14159265359" />
   <xacro:property name="PI_DIV_2" value="1.5707963267948966" />
