Commit message: Add calibration method for sensors based on T pose

File: urdf/human.urdf (robot description, URDF)
Before this commit: robot human_model, 45 links, 44 joints
Links:
- link hip: geometry visual cylinder length=0.0821559601239 radius=0.140925140031
- link left_elbow: geometry visual cylinder length=0.204972218606 radius=0.025
- link left_hip: geometry visual cylinder length=0.514015426058 radius=0.05
- link left_knee: geometry visual cylinder length=0.41640521693 radius=0.025
- link left_shoulder: geometry visual cylinder length=0.280378224637 radius=0.05
- link neck: geometry visual cylinder length=0.19025954166 radius=0.04
- link right_elbow: geometry visual cylinder length=0.204972218606 radius=0.025
- link right_hip: geometry visual cylinder length=0.514015426058 radius=0.05
- link right_knee: geometry visual cylinder length=0.41640521693 radius=0.025
- link right_shoulder: geometry visual cylinder length=0.280378224637 radius=0.05
- link shoulder_center: geometry visual cylinder length=0.0930249603867 radius=0.180925140031
- link spine: geometry visual cylinder length=0.258416861202 radius=0.160925140031
- link waist: geometry visual cylinder length=0.0809381601609 radius=0.160925140031
Joints:
- joint head: origin xyz=0 0 0.184761525418 rpy=0 0 0 -> xyz=0 0 0.19025954166 rpy=0 0 0
- joint left_ankle_0: origin xyz=0.297990595338 0 0 rpy=-1.57079632679 0 1.57079632679 -> xyz=0.41640521693 0 0 rpy=-1.57079632679 0 1.57079632679
- joint left_arm_mount: origin xyz=0 0.17488508899 0 rpy=0 0 1.57079632679 -> xyz=0 0.180925140031 0 rpy=0 0 1.57079632679
- joint left_elbow_0: origin xyz=0.264279890316 0 0 rpy=0 0 0 -> xyz=0.280378224637 0 0 rpy=0 0 0
- joint left_hip_leg_mount: origin xyz=0 0.0729344655435 0 rpy=0 1.57079632679 0 -> xyz=0 0.0762998610903 0 rpy=0 1.57079632679 0
- joint left_knee: origin xyz=0.467551433183 0 0 rpy=1.57079632679 0 0 -> xyz=0.514015426058 0 0 rpy=1.57079632679 0 0
- joint left_wrist_0: origin xyz=0.199200513507 0 0 rpy=0 0 0 -> xyz=0.204972218606 0 0 rpy=0 0 0
- joint neck_0: origin xyz=0 0 0.116117110578 rpy=0 0 0 -> xyz=0 0 0.0930249603867 rpy=0 0 0
- joint right_ankle_0: origin xyz=0.297990595338 0 0 rpy=-1.57079632679 0 1.57079632679 -> xyz=0.41640521693 0 0 rpy=-1.57079632679 0 1.57079632679
- joint right_arm_mount: origin xyz=0 -0.17488508899 0 rpy=0 0 -1.57079632679 -> xyz=0 -0.180925140031 0 rpy=0 0 -1.57079632679
- joint right_elbow_0: origin xyz=0.264279890316 0 0 rpy=0 0 0 -> xyz=0.280378224637 0 0 rpy=0 0 0
- joint right_hip_leg_mount: origin xyz=0 -0.0729344655435 0 rpy=0 1.57079632679 0 -> xyz=0 -0.0762998610903 0 rpy=0 1.57079632679 0
- joint right_knee: origin xyz=0.467551433183 0 0 rpy=1.57079632679 0 0 -> xyz=0.514015426058 0 0 rpy=1.57079632679 0 0
- joint right_wrist_0: origin xyz=0.199200513507 0 0 rpy=0 0 0 -> xyz=0.204972218606 0 0 rpy=0 0 0
- joint shoulder_center: origin xyz=0 0 0.245011240325 rpy=0 0 0 -> xyz=0 0 0.258416861202 rpy=0 0 0
- joint spine: origin xyz=0 0 0.0809393748903 rpy=0 0 0 -> xyz=0 0 0.0809381601609 rpy=0 0 0
- joint waist_0: origin xyz=0 0 0.0790633061127 rpy=0 0 0 -> xyz=0 0 0.0821559601239 rpy=0 0 0

Commit message: Improve calibration of sensor frames
- Add possibility to select frames to be tracked
- Calibration can be performed sensor by sensor

File: urdf/human.urdf (robot description, URDF)
Before this commit: robot human_model, 45 links, 44 joints
Links:
- link hip: geometry visual cylinder length=0.0826712282933 radius=0.144705809145
- link left_elbow: geometry visual cylinder length=0.230486513455 radius=0.025
- link left_hip: geometry visual cylinder length=0.565251792303 radius=0.05
- link left_knee: geometry visual cylinder length=0.349656977126 radius=0.025
- link left_shoulder: geometry visual cylinder length=0.268561323652 radius=0.05
- link neck: geometry visual cylinder length=0.183928282457 radius=0.04
- link right_elbow: geometry visual cylinder length=0.230486513455 radius=0.025
- link right_hip: geometry visual cylinder length=0.565251792303 radius=0.05
- link right_knee: geometry visual cylinder length=0.349656977126 radius=0.025
- link right_shoulder: geometry visual cylinder length=0.268561323652 radius=0.05
- link shoulder_center: geometry visual cylinder length=0.107711169575 radius=0.184705809145
- link spine: geometry visual cylinder length=0.253704151704 radius=0.164705809145
- link waist: geometry visual cylinder length=0.0846063553655 radius=0.164705809145
Joints:
- joint head: origin xyz=0 0 0.19025954166 rpy=0 0 0 -> xyz=0 0 0.183928282457 rpy=0 0 0
- joint left_ankle_0: origin xyz=0.41640521693 0 0 rpy=-1.57079632679 0 1.57079632679 -> xyz=0.349656977126 0 0 rpy=-1.57079632679 0 1.57079632679
- joint left_arm_mount: origin xyz=0 0.180925140031 0 rpy=0 0 1.57079632679 -> xyz=0 0.184705809145 0 rpy=0 0 1.57079632679
- joint left_elbow_0: origin xyz=0.280378224637 0 0 rpy=0 0 0 -> xyz=0.268561323652 0 0 rpy=0 0 0
- joint left_hip_leg_mount: origin xyz=0 0.0762998610903 0 rpy=0 1.57079632679 0 -> xyz=0 0.0813605843123 0 rpy=0 1.57079632679 0
- joint left_knee: origin xyz=0.514015426058 0 0 rpy=1.57079632679 0 0 -> xyz=0.565251792303 0 0 rpy=1.57079632679 0 0
- joint left_wrist_0: origin xyz=0.204972218606 0 0 rpy=0 0 0 -> xyz=0.230486513455 0 0 rpy=0 0 0
- joint neck_0: origin xyz=0 0 0.0930249603867 rpy=0 0 0 -> xyz=0 0 0.107711169575 rpy=0 0 0
- joint right_ankle_0: origin xyz=0.41640521693 0 0 rpy=-1.57079632679 0 1.57079632679 -> xyz=0.349656977126 0 0 rpy=-1.57079632679 0 1.57079632679
- joint right_arm_mount: origin xyz=0 -0.180925140031 0 rpy=0 0 -1.57079632679 -> xyz=0 -0.184705809145 0 rpy=0 0 -1.57079632679
- joint right_elbow_0: origin xyz=0.280378224637 0 0 rpy=0 0 0 -> xyz=0.268561323652 0 0 rpy=0 0 0
- joint right_hip_leg_mount: origin xyz=0 -0.0762998610903 0 rpy=0 1.57079632679 0 -> xyz=0 -0.0813605843123 0 rpy=0 1.57079632679 0
- joint right_knee: origin xyz=0.514015426058 0 0 rpy=1.57079632679 0 0 -> xyz=0.565251792303 0 0 rpy=1.57079632679 0 0
- joint right_wrist_0: origin xyz=0.204972218606 0 0 rpy=0 0 0 -> xyz=0.230486513455 0 0 rpy=0 0 0
- joint shoulder_center: origin xyz=0 0 0.258416861202 rpy=0 0 0 -> xyz=0 0 0.253704151704 rpy=0 0 0
- joint spine: origin xyz=0 0 0.0809381601609 rpy=0 0 0 -> xyz=0 0 0.0846063553655 rpy=0 0 0
- joint waist_0: origin xyz=0 0 0.0821559601239 rpy=0 0 0 -> xyz=0 0 0.0826712282933 rpy=0 0 0

Commit message: Add the possibility to have different ip adress for kinect and optitrack

File: urdf/human.urdf (robot description, URDF)
Before this commit: robot human_model, 45 links, 44 joints
Links:
- link hip: geometry visual cylinder length=0.0812781231253 radius=0.138594483269
- link left_elbow: geometry visual cylinder length=0.226483495078 radius=0.025
- link left_hip: geometry visual cylinder length=0.425049335989 radius=0.05
- link left_knee: geometry visual cylinder length=0.32492779585 radius=0.025
- link left_shoulder: geometry visual cylinder length=0.244728299248 radius=0.05
- link neck: geometry visual cylinder length=0.175502395454 radius=0.04
- link right_elbow: geometry visual cylinder length=0.226483495078 radius=0.025
- link right_hip: geometry visual cylinder length=0.425049335989 radius=0.05
- link right_knee: geometry visual cylinder length=0.32492779585 radius=0.025
- link right_shoulder: geometry visual cylinder length=0.244728299248 radius=0.05
- link shoulder_center: geometry visual cylinder length=0.0994324101673 radius=0.178594483269
- link spine: geometry visual cylinder length=0.247146455532 radius=0.158594483269
- link waist: geometry visual cylinder length=0.0784093271992 radius=0.158594483269
Joints:
- joint head: origin xyz=0 0 0.183928282457 rpy=0 0 0 -> xyz=0 0 0.175502395454 rpy=0 0 0
- joint left_ankle_0: origin xyz=0.349656977126 0 0 rpy=-1.57079632679 0 1.57079632679 -> xyz=0.32492779585 0 0 rpy=-1.57079632679 0 1.57079632679
- joint left_arm_mount: origin xyz=0 0.184705809145 0 rpy=0 0 1.57079632679 -> xyz=0 0.178594483269 0 rpy=0 0 1.57079632679
- joint left_elbow_0: origin xyz=0.268561323652 0 0 rpy=0 0 0 -> xyz=0.244728299248 0 0 rpy=0 0 0
- joint left_hip_leg_mount: origin xyz=0 0.0813605843123 0 rpy=0 1.57079632679 0 -> xyz=0 0.0795324612522 0 rpy=0 1.57079632679 0
- joint left_knee: origin xyz=0.565251792303 0 0 rpy=1.57079632679 0 0 -> xyz=0.425049335989 0 0 rpy=1.57079632679 0 0
- joint left_wrist_0: origin xyz=0.230486513455 0 0 rpy=0 0 0 -> xyz=0.226483495078 0 0 rpy=0 0 0
- joint neck_0: origin xyz=0 0 0.107711169575 rpy=0 0 0 -> xyz=0 0 0.0994324101673 rpy=0 0 0
- joint right_ankle_0: origin xyz=0.349656977126 0 0 rpy=-1.57079632679 0 1.57079632679 -> xyz=0.32492779585 0 0 rpy=-1.57079632679 0 1.57079632679
- joint right_arm_mount: origin xyz=0 -0.184705809145 0 rpy=0 0 -1.57079632679 -> xyz=0 -0.178594483269 0 rpy=0 0 -1.57079632679
- joint right_elbow_0: origin xyz=0.268561323652 0 0 rpy=0 0 0 -> xyz=0.244728299248 0 0 rpy=0 0 0
- joint right_hip_leg_mount: origin xyz=0 -0.0813605843123 0 rpy=0 1.57079632679 0 -> xyz=0 -0.0795324612522 0 rpy=0 1.57079632679 0
- joint right_knee: origin xyz=0.565251792303 0 0 rpy=1.57079632679 0 0 -> xyz=0.425049335989 0 0 rpy=1.57079632679 0 0
- joint right_wrist_0: origin xyz=0.230486513455 0 0 rpy=0 0 0 -> xyz=0.226483495078 0 0 rpy=0 0 0
- joint shoulder_center: origin xyz=0 0 0.253704151704 rpy=0 0 0 -> xyz=0 0 0.247146455532 rpy=0 0 0
- joint spine: origin xyz=0 0 0.0846063553655 rpy=0 0 0 -> xyz=0 0 0.0784093271992 rpy=0 0 0
- joint waist_0: origin xyz=0 0 0.0826712282933 rpy=0 0 0 -> xyz=0 0 0.0812781231253 rpy=0 0 0

Commit message: Remove unused person name argument

File: urdf/human.urdf (robot description, URDF)
Before this commit: robot human_model, 45 links, 44 joints
Links:
- link hip: geometry visual cylinder length=0.0749908293897 radius=0.12869065866
- link left_elbow: geometry visual cylinder length=0.255252770899 radius=0.025
- link left_hip: geometry visual cylinder length=0.458571894166 radius=0.05
- link left_knee: geometry visual cylinder length=0.22800165588 radius=0.025
- link left_shoulder: geometry visual cylinder length=0.255891128261 radius=0.05
- link neck: geometry visual cylinder length=0.149837540981 radius=0.04
- link right_elbow: geometry visual cylinder length=0.255252770899 radius=0.025
- link right_hip: geometry visual cylinder length=0.458571894166 radius=0.05
- link right_knee: geometry visual cylinder length=0.22800165588 radius=0.025
- link right_shoulder: geometry visual cylinder length=0.255891128261 radius=0.05
- link shoulder_center: geometry visual cylinder length=0.0952705796855 radius=0.16869065866
- link spine: geometry visual cylinder length=0.237462362768 radius=0.14869065866
- link waist: geometry visual cylinder length=0.0684808018054 radius=0.14869065866
Joints:
- joint head: origin xyz=0 0 0.175502395454 rpy=0 0 0 -> xyz=0 0 0.149837540981 rpy=0 0 0
- joint left_ankle_0: origin xyz=0.32492779585 0 0 rpy=-1.57079632679 0 1.57079632679 -> xyz=0.22800165588 0 0 rpy=-1.57079632679 0 1.57079632679
- joint left_arm_mount: origin xyz=0 0.178594483269 0 rpy=0 0 1.57079632679 -> xyz=0 0.16869065866 0 rpy=0 0 1.57079632679
- joint left_elbow_0: origin xyz=0.244728299248 0 0 rpy=0 0 0 -> xyz=0.255891128261 0 0 rpy=0 0 0
- joint left_hip_leg_mount: origin xyz=0 0.0795324612522 0 rpy=0 1.57079632679 0 -> xyz=0 0.070480426393 0 rpy=0 1.57079632679 0
- joint left_knee: origin xyz=0.425049335989 0 0 rpy=1.57079632679 0 0 -> xyz=0.458571894166 0 0 rpy=1.57079632679 0 0
- joint left_wrist_0: origin xyz=0.226483495078 0 0 rpy=0 0 0 -> xyz=0.255252770899 0 0 rpy=0 0 0
- joint neck_0: origin xyz=0 0 0.0994324101673 rpy=0 0 0 -> xyz=0 0 0.0952705796855 rpy=0 0 0
- joint right_ankle_0: origin xyz=0.32492779585 0 0 rpy=-1.57079632679 0 1.57079632679 -> xyz=0.22800165588 0 0 rpy=-1.57079632679 0 1.57079632679
- joint right_arm_mount: origin xyz=0 -0.178594483269 0 rpy=0 0 -1.57079632679 -> xyz=0 -0.16869065866 0 rpy=0 0 -1.57079632679
- joint right_elbow_0: origin xyz=0.244728299248 0 0 rpy=0 0 0 -> xyz=0.255891128261 0 0 rpy=0 0 0
- joint right_hip_leg_mount: origin xyz=0 -0.0795324612522 0 rpy=0 1.57079632679 0 -> xyz=0 -0.070480426393 0 rpy=0 1.57079632679 0
- joint right_knee: origin xyz=0.425049335989 0 0 rpy=1.57079632679 0 0 -> xyz=0.458571894166 0 0 rpy=1.57079632679 0 0
- joint right_wrist_0: origin xyz=0.226483495078 0 0 rpy=0 0 0 -> xyz=0.255252770899 0 0 rpy=0 0 0
- joint shoulder_center: origin xyz=0 0 0.247146455532 rpy=0 0 0 -> xyz=0 0 0.237462362768 rpy=0 0 0
- joint spine: origin xyz=0 0 0.0784093271992 rpy=0 0 0 -> xyz=0 0 0.0684808018054 rpy=0 0 0
- joint waist_0: origin xyz=0 0 0.0812781231253 rpy=0 0 0 -> xyz=0 0 0.0749908293897 rpy=0 0 0

Commit message: update model for kinect 2 usage

File: urdf/human.urdf (robot description, URDF)
Before this commit: robot human_model, 45 links, 44 joints
Links:
- removed link hip
- removed link waist
- removed link waist_0
- removed link waist_1
- added link spine_0; visual cylinder length=0.0791883416579 radius=0.153709147861
- added link spine_1
- added link spine_2
- link base: geometry visual cylinder length=-0.082907600998 radius=0.132513648175
- link left_elbow: geometry visual cylinder length=0.22785848249 radius=0.025
- link left_hip: geometry visual cylinder length=0.413723532258 radius=0.05
- link left_knee: geometry visual cylinder length=0.286981751016 radius=0.025
- link left_shoulder: geometry visual cylinder length=0.284485147659 radius=0.05
- link neck: geometry visual cylinder length=0.196534765643 radius=0.04
- link right_elbow: geometry visual cylinder length=0.22785848249 radius=0.025
- link right_hip: geometry visual cylinder length=0.413723532258 radius=0.05
- link right_knee: geometry visual cylinder length=0.286981751016 radius=0.025
- link right_shoulder: geometry visual cylinder length=0.284485147659 radius=0.05
- link shoulder_center: geometry visual cylinder length=0.0938357552317 radius=0.193709147861
- link spine: geometry visual cylinder length=0.246614217729 radius=0.173709147861
Joints:
- removed joint spine
- removed joint waist_0
- removed joint waist_1
- removed joint waist_2
- added joint spine_0: type revolute, parent spine_0, child spine_1, origin xyz=0 0 0.0791883416579 rpy=0 0 0, axis 1 0 0, limit lower=-1.57079632679 upper=1.57079632679 effort=1 velocity=1
- added joint spine_1: type revolute, parent spine_1, child spine_2, origin xyz=0 0 0 rpy=0 0 0, axis 0 1 0, limit lower=-1.57079632679 upper=1.57079632679 effort=1 velocity=1
- added joint spine_2: type revolute, parent spine_2, child spine, origin xyz=0 0 0 rpy=0 0 0, axis 0 0 1, limit lower=-1.57079632679 upper=1.57079632679 effort=1 velocity=1
- joint head: origin xyz=0 0 0.149837540981 rpy=0 0 0 -> xyz=0 0 0.196534765643 rpy=0 0 0
- joint hip: child hip -> spine_0
- joint left_ankle_0: origin xyz=0.22800165588 0 0 rpy=-1.57079632679 0 1.57079632679 -> xyz=0.286981751016 0 0 rpy=-1.57079632679 0 1.57079632679
- joint left_arm_mount: origin xyz=0 0.16869065866 0 rpy=0 0 1.57079632679 -> xyz=0 0.193709147861 0.000434874900946 rpy=0 0 1.57079632679
- joint left_elbow_0: origin xyz=0.255891128261 0 0 rpy=0 0 0 -> xyz=0.284485147659 0 0 rpy=0 0 0
- joint left_hip_leg_mount: origin xyz=0 0.070480426393 0 rpy=0 1.57079632679 0 -> xyz=0 0.0825136481749 -0.082907600998 rpy=0 1.57079632679 0
- joint left_knee: origin xyz=0.458571894166 0 0 rpy=1.57079632679 0 0 -> xyz=0.413723532258 0 0 rpy=1.57079632679 0 0
- joint left_wrist_0: origin xyz=0.255252770899 0 0 rpy=0 0 0 -> xyz=0.22785848249 0 0 rpy=0 0 0
- joint neck_0: origin xyz=0 0 0.0952705796855 rpy=0 0 0 -> xyz=0 0 0.0938357552317 rpy=0 0 0
- joint right_ankle_0: origin xyz=0.22800165588 0 0 rpy=-1.57079632679 0 1.57079632679 -> xyz=0.286981751016 0 0 rpy=-1.57079632679 0 1.57079632679
- joint right_arm_mount: origin xyz=0 -0.16869065866 0 rpy=0 0 -1.57079632679 -> xyz=0 -0.193709147861 0.000434874900946 rpy=0 0 -1.57079632679
- joint right_elbow_0: origin xyz=0.255891128261 0 0 rpy=0 0 0 -> xyz=0.284485147659 0 0 rpy=0 0 0
- joint right_hip_leg_mount: origin xyz=0 -0.070480426393 0 rpy=0 1.57079632679 0 -> xyz=0 -0.0825136481749 -0.082907600998 rpy=0 1.57079632679 0
- joint right_knee: origin xyz=0.458571894166 0 0 rpy=1.57079632679 0 0 -> xyz=0.413723532258 0 0 rpy=1.57079632679 0 0
- joint right_wrist_0: origin xyz=0.255252770899 0 0 rpy=0 0 0 -> xyz=0.22785848249 0 0 rpy=0 0 0
- joint shoulder_center: origin xyz=0 0 0.237462362768 rpy=0 0 0 -> xyz=0 0 0.246614217729 rpy=0 0 0

File: urdf/xacro/human_arm.urdf.xacro (robot description, xacro)
@@ -35,5 +35,5 @@
     <!-- Joints -->
     <joint name="${side}_arm_mount" type="fixed">
-      <origin xyz="0 ${reflect*shoulder_offset_width} 0" rpy="0 0 ${reflect*PI_DIV_2}" />
+      <origin xyz="0 ${reflect*shoulder_offset_width} ${shoulder_offset_height}" rpy="0 0 ${reflect*PI_DIV_2}" />
       <parent link="shoulder_center" />
       <child link="${side}_arm_mount" />

File: urdf/xacro/human_body.urdf.xacro (robot description, xacro)
@@ -3,31 +3,27 @@
 <xacro:include filename="props_global.urdf.xacro" />
 <xacro:macro name="human_body">
-	<link name="base"/>
-    <link name="hip">
+	  <link name="base">
       <visual>
-        <origin xyz="0 0 ${waist_length/2}" rpy="0 0 0" />
+        <origin xyz="0 0 ${-hip_offset_height/2}" rpy="0 0 0" />
         <geometry>
-          <!--<box size="0.4 0.2 ${waist_length}" />-->
-          <cylinder radius="${waist_radius}" length="${waist_length}" />
+          <cylinder radius="${hip_offset_width+thigh_radius}" length="${-hip_offset_height}" />
         </geometry>
       </visual>
     </link>
-    <link name="waist_0"/>
-    <link name="waist_1"/>
-    <link name="waist">
+    <link name="spine_0">
       <visual>
         <origin xyz="0 0 ${spine_down_length/2}" rpy="0 0 0" />
         <geometry>
-          <!--<box size="0.4 0.2 ${torso_length}" />-->
-          <cylinder radius="${spine_radius}" length="${spine_down_length}" />
+          <cylinder radius="${spine_down_radius}" length="${spine_down_length}" />
         </geometry>
       </visual>
     </link>
+    <link name="spine_1"/>
+    <link name="spine_2"/>
     <link name="spine">
       <visual>
         <origin xyz="0 0 ${spine_up_length/2}" rpy="0 0 0" />
         <geometry>
-	        <!--<box size="0.4 0.2 ${torso_length}" />-->
-	        <cylinder radius="${spine_radius}" length="${spine_up_length}" />
+          <cylinder radius="${spine_up_radius}" length="${spine_up_length}" />
         </geometry>
       </visual>
@@ -37,5 +33,4 @@
         <origin xyz="0 0 ${torso_length/2}" rpy="0 0 0" />
         <geometry>
-          <!--<box size="0.4 0.2 ${torso_length}" />-->
           <cylinder radius="${torso_radius}" length="${torso_length}" />
         </geometry>
@@ -48,5 +43,4 @@
         <origin xyz="0 0 ${neck_length/2}" rpy="0 0 0" />
         <geometry>
-          <!--<box size="0.4 0.2 ${torso_length}" />-->
           <cylinder radius="${neck_radius}" length="${neck_length}" />
         </geometry>
@@ -64,32 +58,25 @@
       <origin xyz="0 0 0" rpy="0 0 0" />
       <parent link="base" />
-      <child link="hip" />
+      <child link="spine_0" />
     </joint>
     <!-- SPINE : spherical -->
-    <joint name="waist_0" type="revolute">
-      <origin xyz="0 0 ${waist_length}" rpy="0 0 0" />
+    <joint name="spine_0" type="revolute">
+      <origin xyz="0 0 ${spine_down_length}" rpy="0 0 0" />
       <axis xyz="1 0 0" />
-      <parent link="hip" />
-      <child link="waist_0" />
+      <parent link="spine_0" />
+      <child link="spine_1" />
       <limit lower="${-PI_DIV_2}" upper="${PI_DIV_2}" effort="${max_effort}" velocity="${max_velocity}" />
     </joint>
-    <joint name="waist_1" type="revolute">
+    <joint name="spine_1" type="revolute">
       <origin xyz="0 0 0" rpy="0 0 0" />
       <axis xyz="0 1 0" />
-      <parent link="waist_0" />
-      <child link="waist_1" />
+      <parent link="spine_1" />
+      <child link="spine_2" />
       <limit lower="${-PI_DIV_2}" upper="${PI_DIV_2}" effort="${max_effort}" velocity="${max_velocity}" />
     </joint>
-    <joint name="waist_2" type="revolute">
+    <joint name="spine_2" type="revolute">
       <origin xyz="0 0 0" rpy="0 0 0" />
       <axis xyz="0 0 1" />
-      <parent link="waist_1" />
-      <child link="waist" />
-      <limit lower="${-PI_DIV_2}" upper="${PI_DIV_2}" effort="${max_effort}" velocity="${max_velocity}" />
-    </joint>
-    <joint name="spine" type="revolute">
-      <origin xyz="0 0 ${spine_down_length}" rpy="0 0 0" />
-      <axis xyz="0 1 0" />
-      <parent link="waist" />
+      <parent link="spine_2" />
       <child link="spine" />
       <limit lower="${-PI_DIV_2}" upper="${PI_DIV_2}" effort="${max_effort}" velocity="${max_velocity}" />

File: urdf/xacro/human_leg.urdf.xacro (robot description, xacro)
@@ -10,5 +10,5 @@
         <origin xyz="${thigh_length/2} 0 0" rpy="0 ${PI_DIV_2} 0" />
         <geometry>
-	        <cylinder radius="0.05" length="${thigh_length}" />
+	        <cylinder radius="${thigh_radius}" length="${thigh_length}" />
         </geometry>
       </visual>
@@ -34,5 +34,5 @@
     <!-- Joints -->
     <joint name="${side}_hip_leg_mount" type="fixed">
-      <origin xyz="0 ${reflect*hip_offset_width} 0" rpy="0 ${PI_DIV_2} 0" />
+      <origin xyz="0 ${reflect*hip_offset_width} ${-hip_offset_height}" rpy="0 ${PI_DIV_2} 0" />
       <parent link="base" />
       <child link="${side}_leg_mount" />

File: urdf/xacro/props_global.urdf.xacro (robot description, xacro)
@@ -15,16 +15,18 @@
   <xacro:property name="torso_length" value="$(arg torso_length)" />
   <xacro:property name="torso_radius" value="$(arg torso_radius)" />
-  <xacro:property name="waist_length" value="$(arg waist_length)" />
-  <xacro:property name="waist_radius" value="$(arg waist_radius)" />
   <xacro:property name="spine_down_length" value="$(arg spine_down_length)" />
   <xacro:property name="spine_up_length" value="$(arg spine_up_length)" />
-  <xacro:property name="spine_radius" value="$(arg spine_radius)" />
+  <xacro:property name="spine_down_radius" value="$(arg spine_down_radius)" />
+  <xacro:property name="spine_up_radius" value="$(arg spine_up_radius)" />
   <xacro:property name="neck_length" value="$(arg neck_length)" />
   <xacro:property name="neck_radius" value="$(arg neck_radius)" />
   <xacro:property name="thigh_length" value="$(arg thigh_length)" />
+  <xacro:property name="thigh_radius" value="$(arg thigh_radius)" />
   <xacro:property name="shin_length" value="$(arg shin_length)" />
   <xacro:property name="foot_length" value="$(arg foot_length)" />
   <xacro:property name="shoulder_offset_width" value="$(arg shoulder_offset_width)" />
+  <xacro:property name="shoulder_offset_height" value="$(arg shoulder_offset_height)" />
   <xacro:property name="hip_offset_width" value="$(arg hip_offset_width)" />
+  <xacro:property name="hip_offset_height" value="$(arg hip_offset_height)" />
   <xacro:property name="max_effort" value="1" />
   <xacro:property name="max_velocity" value="1" />
