Commit message: Add file of permutations

File: urdf/human.urdf (robot description, URDF)
Before this commit: robot human_model, 44 links, 43 joints
Links:
- link base: geometry visual cylinder length=-0.0849158933353 radius=0.124021830901
- link left_elbow: geometry visual cylinder length=0.208975034701 radius=0.025
- link left_hip: geometry visual cylinder length=0.461369870064 radius=0.05
- link left_knee: geometry visual cylinder length=0.276082487516 radius=0.025
- link left_shoulder: geometry visual cylinder length=0.251684860572 radius=0.05
- link neck: geometry visual cylinder length=0.188740765099 radius=0.04
- link right_elbow: geometry visual cylinder length=0.208975034701 radius=0.025
- link right_hip: geometry visual cylinder length=0.461369870064 radius=0.05
- link right_knee: geometry visual cylinder length=0.276082487516 radius=0.025
- link right_shoulder: geometry visual cylinder length=0.251684860572 radius=0.05
- link shoulder_center: geometry visual cylinder length=0.0960913366537 radius=0.192957195419
- link spine: geometry visual cylinder length=0.225559264046 radius=0.172957195419
- link spine_0: geometry visual cylinder length=0.0749147887744 radius=0.152957195419
Joints:
- joint head: origin xyz=0 0 0.196534765643 rpy=0 0 0 -> xyz=0 0 0.188740765099 rpy=0 0 0
- joint left_ankle_0: origin xyz=0.286981751016 0 0 rpy=-1.57079632679 0 1.57079632679 -> xyz=0.276082487516 0 0 rpy=-1.57079632679 0 1.57079632679
- joint left_arm_mount: origin xyz=0 0.193709147861 0.000434874900946 rpy=0 0 1.57079632679 -> xyz=0 0.192957195419 -0.00377962265178 rpy=0 0 1.57079632679
- joint left_elbow_0: origin xyz=0.284485147659 0 0 rpy=0 0 0 -> xyz=0.251684860572 0 0 rpy=0 0 0
- joint left_hip_leg_mount: origin xyz=0 0.0825136481749 -0.082907600998 rpy=0 1.57079632679 0 -> xyz=0 0.074021830901 -0.0849158933353 rpy=0 1.57079632679 0
- joint left_knee: origin xyz=0.413723532258 0 0 rpy=1.57079632679 0 0 -> xyz=0.461369870064 0 0 rpy=1.57079632679 0 0
- joint left_wrist_0: origin xyz=0.22785848249 0 0 rpy=0 0 0 -> xyz=0.208975034701 0 0 rpy=0 0 0
- joint neck_0: origin xyz=0 0 0.0938357552317 rpy=0 0 0 -> xyz=0 0 0.0960913366537 rpy=0 0 0
- joint right_ankle_0: origin xyz=0.286981751016 0 0 rpy=-1.57079632679 0 1.57079632679 -> xyz=0.276082487516 0 0 rpy=-1.57079632679 0 1.57079632679
- joint right_arm_mount: origin xyz=0 -0.193709147861 0.000434874900946 rpy=0 0 -1.57079632679 -> xyz=0 -0.192957195419 -0.00377962265178 rpy=0 0 -1.57079632679
- joint right_elbow_0: origin xyz=0.284485147659 0 0 rpy=0 0 0 -> xyz=0.251684860572 0 0 rpy=0 0 0
- joint right_hip_leg_mount: origin xyz=0 -0.0825136481749 -0.082907600998 rpy=0 1.57079632679 0 -> xyz=0 -0.074021830901 -0.0849158933353 rpy=0 1.57079632679 0
- joint right_knee: origin xyz=0.413723532258 0 0 rpy=1.57079632679 0 0 -> xyz=0.461369870064 0 0 rpy=1.57079632679 0 0
- joint right_wrist_0: origin xyz=0.22785848249 0 0 rpy=0 0 0 -> xyz=0.208975034701 0 0 rpy=0 0 0
- joint shoulder_center: origin xyz=0 0 0.246614217729 rpy=0 0 0 -> xyz=0 0 0.225559264046 rpy=0 0 0
- joint spine_0: origin xyz=0 0 0.0791883416579 rpy=0 0 0 -> xyz=0 0 0.0749147887744 rpy=0 0 0

Commit message: Changes names of robot state and joint state publisher
Default names were also used by Baxter. Rename nodes to avoid conflict

File: urdf/human.urdf (robot description, URDF)
Before this commit: robot human_model, 44 links, 43 joints
Links:
- link base: geometry visual cylinder length=-0.0873286156238 radius=0.13032805021
- link left_elbow: geometry visual cylinder length=0.240598707909 radius=0.025
- link left_hip: geometry visual cylinder length=0.579184611426 radius=0.05
- link left_knee: geometry visual cylinder length=0.378014044036 radius=0.025
- link left_shoulder: geometry visual cylinder length=0.263302375161 radius=0.05
- link neck: geometry visual cylinder length=0.186621149291 radius=0.04
- link right_elbow: geometry visual cylinder length=0.240598707909 radius=0.025
- link right_hip: geometry visual cylinder length=0.579184611426 radius=0.05
- link right_knee: geometry visual cylinder length=0.378014044036 radius=0.025
- link right_shoulder: geometry visual cylinder length=0.263302375161 radius=0.05
- link shoulder_center: geometry visual cylinder length=0.0787097042481 radius=0.193572664486
- link spine: geometry visual cylinder length=0.271570566311 radius=0.173572664486
- link spine_0: geometry visual cylinder length=0.0711357524669 radius=0.153572664486
Joints:
- joint head: origin xyz=0 0 0.188740765099 rpy=0 0 0 -> xyz=0 0 0.186621149291 rpy=0 0 0
- joint left_ankle_0: origin xyz=0.276082487516 0 0 rpy=-1.57079632679 0 1.57079632679 -> xyz=0.378014044036 0 0 rpy=-1.57079632679 0 1.57079632679
- joint left_arm_mount: origin xyz=0 0.192957195419 -0.00377962265178 rpy=0 0 1.57079632679 -> xyz=0 0.193572664486 -0.00334000635564 rpy=0 0 1.57079632679
- joint left_elbow_0: origin xyz=0.251684860572 0 0 rpy=0 0 0 -> xyz=0.263302375161 0 0 rpy=0 0 0
- joint left_hip_leg_mount: origin xyz=0 0.074021830901 -0.0849158933353 rpy=0 1.57079632679 0 -> xyz=0 0.0803280502102 -0.0873286156238 rpy=0 1.57079632679 0
- joint left_knee: origin xyz=0.461369870064 0 0 rpy=1.57079632679 0 0 -> xyz=0.579184611426 0 0 rpy=1.57079632679 0 0
- joint left_wrist_0: origin xyz=0.208975034701 0 0 rpy=0 0 0 -> xyz=0.240598707909 0 0 rpy=0 0 0
- joint neck_0: origin xyz=0 0 0.0960913366537 rpy=0 0 0 -> xyz=0 0 0.0787097042481 rpy=0 0 0
- joint right_ankle_0: origin xyz=0.276082487516 0 0 rpy=-1.57079632679 0 1.57079632679 -> xyz=0.378014044036 0 0 rpy=-1.57079632679 0 1.57079632679
- joint right_arm_mount: origin xyz=0 -0.192957195419 -0.00377962265178 rpy=0 0 -1.57079632679 -> xyz=0 -0.193572664486 -0.00334000635564 rpy=0 0 -1.57079632679
- joint right_elbow_0: origin xyz=0.251684860572 0 0 rpy=0 0 0 -> xyz=0.263302375161 0 0 rpy=0 0 0
- joint right_hip_leg_mount: origin xyz=0 -0.074021830901 -0.0849158933353 rpy=0 1.57079632679 0 -> xyz=0 -0.0803280502102 -0.0873286156238 rpy=0 1.57079632679 0
- joint right_knee: origin xyz=0.461369870064 0 0 rpy=1.57079632679 0 0 -> xyz=0.579184611426 0 0 rpy=1.57079632679 0 0
- joint right_wrist_0: origin xyz=0.208975034701 0 0 rpy=0 0 0 -> xyz=0.240598707909 0 0 rpy=0 0 0
- joint shoulder_center: origin xyz=0 0 0.225559264046 rpy=0 0 0 -> xyz=0 0 0.271570566311 rpy=0 0 0
- joint spine_0: origin xyz=0 0 0.0749147887744 rpy=0 0 0 -> xyz=0 0 0.0711357524669 rpy=0 0 0

Commit message: Add a boolean to launch the kinect_skeleton_publisher only when necessary

File: urdf/human.urdf (robot description, URDF)
Before this commit: robot human_model, 44 links, 43 joints
Links:
- link base: geometry visual cylinder length=-0.0829335515941 radius=0.132940409993
- link left_elbow: geometry visual cylinder length=0.243174868618 radius=0.025
- link left_hip: geometry visual cylinder length=0.493353757924 radius=0.05
- link left_knee: geometry visual cylinder length=0.44903502583 radius=0.025
- link left_shoulder: geometry visual cylinder length=0.329208547146 radius=0.05
- link neck: geometry visual cylinder length=0.176471493454 radius=0.04
- link right_elbow: geometry visual cylinder length=0.243174868618 radius=0.025
- link right_hip: geometry visual cylinder length=0.493353757924 radius=0.05
- link right_knee: geometry visual cylinder length=0.44903502583 radius=0.025
- link right_shoulder: geometry visual cylinder length=0.329208547146 radius=0.05
- link shoulder_center: geometry visual cylinder length=0.0904162732757 radius=0.186690880778
- link spine: geometry visual cylinder length=0.278219894477 radius=0.166690880778
- link spine_0: geometry visual cylinder length=0.0740256374914 radius=0.146690880778
Joints:
- joint head: origin xyz=0 0 0.186621149291 rpy=0 0 0 -> xyz=0 0 0.176471493454 rpy=0 0 0
- joint left_ankle_0: origin xyz=0.378014044036 0 0 rpy=-1.57079632679 0 1.57079632679 -> xyz=0.44903502583 0 0 rpy=-1.57079632679 0 1.57079632679
- joint left_arm_mount: origin xyz=0 0.193572664486 -0.00334000635564 rpy=0 0 1.57079632679 -> xyz=0 0.186690880778 0.00504378778975 rpy=0 0 1.57079632679
- joint left_elbow_0: origin xyz=0.263302375161 0 0 rpy=0 0 0 -> xyz=0.329208547146 0 0 rpy=0 0 0
- joint left_hip_leg_mount: origin xyz=0 0.0803280502102 -0.0873286156238 rpy=0 1.57079632679 0 -> xyz=0 0.0829404099932 -0.0829335515941 rpy=0 1.57079632679 0
- joint left_knee: origin xyz=0.579184611426 0 0 rpy=1.57079632679 0 0 -> xyz=0.493353757924 0 0 rpy=1.57079632679 0 0
- joint left_wrist_0: origin xyz=0.240598707909 0 0 rpy=0 0 0 -> xyz=0.243174868618 0 0 rpy=0 0 0
- joint neck_0: origin xyz=0 0 0.0787097042481 rpy=0 0 0 -> xyz=0 0 0.0904162732757 rpy=0 0 0
- joint right_ankle_0: origin xyz=0.378014044036 0 0 rpy=-1.57079632679 0 1.57079632679 -> xyz=0.44903502583 0 0 rpy=-1.57079632679 0 1.57079632679
- joint right_arm_mount: origin xyz=0 -0.193572664486 -0.00334000635564 rpy=0 0 -1.57079632679 -> xyz=0 -0.186690880778 0.00504378778975 rpy=0 0 -1.57079632679
- joint right_elbow_0: origin xyz=0.263302375161 0 0 rpy=0 0 0 -> xyz=0.329208547146 0 0 rpy=0 0 0
- joint right_hip_leg_mount: origin xyz=0 -0.0803280502102 -0.0873286156238 rpy=0 1.57079632679 0 -> xyz=0 -0.0829404099932 -0.0829335515941 rpy=0 1.57079632679 0
- joint right_knee: origin xyz=0.579184611426 0 0 rpy=1.57079632679 0 0 -> xyz=0.493353757924 0 0 rpy=1.57079632679 0 0
- joint right_wrist_0: origin xyz=0.240598707909 0 0 rpy=0 0 0 -> xyz=0.243174868618 0 0 rpy=0 0 0
- joint shoulder_center: origin xyz=0 0 0.271570566311 rpy=0 0 0 -> xyz=0 0 0.278219894477 rpy=0 0 0
- joint spine_0: origin xyz=0 0 0.0711357524669 rpy=0 0 0 -> xyz=0 0 0.0740256374914 rpy=0 0 0

Commit message: Major changes in the optitrack calibration
- Changes the torso marker to be fit on the shoulder_center instead of
the spine frame. This has required to also change the namespace
"/optitrack" to "/opt" as the marker name
"/optitrack/human/shoulder_center" is too long for motive to handle.

- Add a verification on the initial base frame guess for the
optimization such that x base axis always face the robot. This handles
cases were the initial guess was facing opposite which lead to not
converging calibration

File: urdf/human.urdf (robot description, URDF)
Before this commit: robot human_model, 44 links, 43 joints
Links:
- link base: geometry visual cylinder length=-0.0926440214385 radius=0.127898794835
- link left_elbow: geometry visual cylinder length=0.239489837596 radius=0.025
- link left_hip: geometry visual cylinder length=0.56353659918 radius=0.05
- link left_knee: geometry visual cylinder length=0.427367160654 radius=0.025
- link left_shoulder: geometry visual cylinder length=0.297734734429 radius=0.05
- link neck: geometry visual cylinder length=0.192881539905 radius=0.04
- link right_elbow: geometry visual cylinder length=0.239489837596 radius=0.025
- link right_hip: geometry visual cylinder length=0.56353659918 radius=0.05
- link right_knee: geometry visual cylinder length=0.427367160654 radius=0.025
- link right_shoulder: geometry visual cylinder length=0.297734734429 radius=0.05
- link shoulder_center: geometry visual cylinder length=0.117065294255 radius=0.208266491877
- link spine: geometry visual cylinder length=0.24974378696 radius=0.188266491877
- link spine_0: geometry visual cylinder length=0.0868936531215 radius=0.168266491877
Joints:
- joint head: origin xyz=0 0 0.176471493454 rpy=0 0 0 -> xyz=0 0 0.192881539905 rpy=0 0 0
- joint left_ankle_0: origin xyz=0.44903502583 0 0 rpy=-1.57079632679 0 1.57079632679 -> xyz=0.427367160654 0 0 rpy=-1.57079632679 0 1.57079632679
- joint left_arm_mount: origin xyz=0 0.186690880778 0.00504378778975 rpy=0 0 1.57079632679 -> xyz=0 0.208266491877 -0.000734663379099 rpy=0 0 1.57079632679
- joint left_elbow_0: origin xyz=0.329208547146 0 0 rpy=0 0 0 -> xyz=0.297734734429 0 0 rpy=0 0 0
- joint left_hip_leg_mount: origin xyz=0 0.0829404099932 -0.0829335515941 rpy=0 1.57079632679 0 -> xyz=0 0.0778987948353 -0.0926440214385 rpy=0 1.57079632679 0
- joint left_knee: origin xyz=0.493353757924 0 0 rpy=1.57079632679 0 0 -> xyz=0.56353659918 0 0 rpy=1.57079632679 0 0
- joint left_wrist_0: origin xyz=0.243174868618 0 0 rpy=0 0 0 -> xyz=0.239489837596 0 0 rpy=0 0 0
- joint neck_0: origin xyz=0 0 0.0904162732757 rpy=0 0 0 -> xyz=0 0 0.117065294255 rpy=0 0 0
- joint right_ankle_0: origin xyz=0.44903502583 0 0 rpy=-1.57079632679 0 1.57079632679 -> xyz=0.427367160654 0 0 rpy=-1.57079632679 0 1.57079632679
- joint right_arm_mount: origin xyz=0 -0.186690880778 0.00504378778975 rpy=0 0 -1.57079632679 -> xyz=0 -0.208266491877 -0.000734663379099 rpy=0 0 -1.57079632679
- joint right_elbow_0: origin xyz=0.329208547146 0 0 rpy=0 0 0 -> xyz=0.297734734429 0 0 rpy=0 0 0
- joint right_hip_leg_mount: origin xyz=0 -0.0829404099932 -0.0829335515941 rpy=0 1.57079632679 0 -> xyz=0 -0.0778987948353 -0.0926440214385 rpy=0 1.57079632679 0
- joint right_knee: origin xyz=0.493353757924 0 0 rpy=1.57079632679 0 0 -> xyz=0.56353659918 0 0 rpy=1.57079632679 0 0
- joint right_wrist_0: origin xyz=0.243174868618 0 0 rpy=0 0 0 -> xyz=0.239489837596 0 0 rpy=0 0 0
- joint shoulder_center: origin xyz=0 0 0.278219894477 rpy=0 0 0 -> xyz=0 0 0.24974378696 rpy=0 0 0
- joint spine_0: origin xyz=0 0 0.0740256374914 rpy=0 0 0 -> xyz=0 0 0.0868936531215 rpy=0 0 0

Commit message: new urdf version

File: urdf/human.urdf (robot description, URDF)
Before this commit: robot human_model, 44 links, 43 joints
Links:
- link base: geometry visual cylinder length=-0.0855449172121 radius=0.132393216828
- link left_elbow: geometry visual cylinder length=0.241500492953 radius=0.025
- link left_hip: geometry visual cylinder length=0.599774544438 radius=0.05
- link left_knee: geometry visual cylinder length=0.377295708046 radius=0.025
- link left_shoulder: geometry visual cylinder length=0.298109797064 radius=0.05
- link neck: geometry visual cylinder length=0.194702136255 radius=0.04
- link right_elbow: geometry visual cylinder length=0.241500492953 radius=0.025
- link right_hip: geometry visual cylinder length=0.599774544438 radius=0.05
- link right_knee: geometry visual cylinder length=0.377295708046 radius=0.025
- link right_shoulder: geometry visual cylinder length=0.298109797064 radius=0.05
- link shoulder_center: geometry visual cylinder length=0.105622495203 radius=0.19918889412
- link spine: geometry visual cylinder length=0.249607579586 radius=0.17918889412
- link spine_0: geometry visual cylinder length=0.0838337572759 radius=0.15918889412
Joints:
- joint head: origin xyz=0 0 0.192881539905 rpy=0 0 0 -> xyz=0 0 0.194702136255 rpy=0 0 0
- joint left_ankle_0: origin xyz=0.427367160654 0 0 rpy=-1.57079632679 0 1.57079632679 -> xyz=0.377295708046 0 0 rpy=-1.57079632679 0 1.57079632679
- joint left_arm_mount: origin xyz=0 0.208266491877 -0.000734663379099 rpy=0 0 1.57079632679 -> xyz=0 0.19918889412 0.00217313207535 rpy=0 0 1.57079632679
- joint left_elbow_0: origin xyz=0.297734734429 0 0 rpy=0 0 0 -> xyz=0.298109797064 0 0 rpy=0 0 0
- joint left_hip_leg_mount: origin xyz=0 0.0778987948353 -0.0926440214385 rpy=0 1.57079632679 0 -> xyz=0 0.0823932168285 -0.0855449172121 rpy=0 1.57079632679 0
- joint left_knee: origin xyz=0.56353659918 0 0 rpy=1.57079632679 0 0 -> xyz=0.599774544438 0 0 rpy=1.57079632679 0 0
- joint left_wrist_0: origin xyz=0.239489837596 0 0 rpy=0 0 0 -> xyz=0.241500492953 0 0 rpy=0 0 0
- joint neck_0: origin xyz=0 0 0.117065294255 rpy=0 0 0 -> xyz=0 0 0.105622495203 rpy=0 0 0
- joint right_ankle_0: origin xyz=0.427367160654 0 0 rpy=-1.57079632679 0 1.57079632679 -> xyz=0.377295708046 0 0 rpy=-1.57079632679 0 1.57079632679
- joint right_arm_mount: origin xyz=0 -0.208266491877 -0.000734663379099 rpy=0 0 -1.57079632679 -> xyz=0 -0.19918889412 0.00217313207535 rpy=0 0 -1.57079632679
- joint right_elbow_0: origin xyz=0.297734734429 0 0 rpy=0 0 0 -> xyz=0.298109797064 0 0 rpy=0 0 0
- joint right_hip_leg_mount: origin xyz=0 -0.0778987948353 -0.0926440214385 rpy=0 1.57079632679 0 -> xyz=0 -0.0823932168285 -0.0855449172121 rpy=0 1.57079632679 0
- joint right_knee: origin xyz=0.56353659918 0 0 rpy=1.57079632679 0 0 -> xyz=0.599774544438 0 0 rpy=1.57079632679 0 0
- joint right_wrist_0: origin xyz=0.239489837596 0 0 rpy=0 0 0 -> xyz=0.241500492953 0 0 rpy=0 0 0
- joint shoulder_center: origin xyz=0 0 0.24974378696 rpy=0 0 0 -> xyz=0 0 0.249607579586 rpy=0 0 0
- joint spine_0: origin xyz=0 0 0.0868936531215 rpy=0 0 0 -> xyz=0 0 0.0838337572759 rpy=0 0 0
