Commit message: Add a prefix to each link of the URDF to avoid conflicts with Baxter

File: urdf/human.urdf (robot description, URDF)
Before this commit: robot human_model, 44 links, 43 joints
Links:
- removed link base
- removed link head
- removed link left_ankle
- removed link left_ankle_0
- removed link left_arm_mount
- removed link left_elbow
- removed link left_elbow_0
- removed link left_foot
- removed link left_hand
- removed link left_hip
- removed link left_hip_0
- removed link left_hip_1
- removed link left_knee
- removed link left_leg_mount
- removed link left_shoulder
- removed link left_shoulder_0
- removed link left_shoulder_1
- removed link left_wrist
- removed link left_wrist_0
- removed link neck
- removed link neck_0
- removed link neck_1
- removed link right_ankle
- removed link right_ankle_0
- removed link right_arm_mount
- removed link right_elbow
- removed link right_elbow_0
- removed link right_foot
- removed link right_hand
- removed link right_hip
- removed link right_hip_0
- removed link right_hip_1
- removed link right_knee
- removed link right_leg_mount
- removed link right_shoulder
- removed link right_shoulder_0
- removed link right_shoulder_1
- removed link right_wrist
- removed link right_wrist_0
- removed link shoulder_center
- removed link spine
- removed link spine_0
- removed link spine_1
- removed link spine_2
- added link /human/base; visual cylinder length=-0.106054276781 radius=0.119385830463
- added link /human/head; visual sphere radius=0.1
- added link /human/left_ankle; visual box size=0.1 0.05 .005
- added link /human/left_ankle_0
- added link /human/left_arm_mount
- added link /human/left_elbow; visual cylinder length=0.226603262858 radius=0.025
- added link /human/left_elbow_0
- added link /human/left_foot
- added link /human/left_hand
- added link /human/left_hip; visual cylinder length=0.366580233013 radius=0.05
- added link /human/left_hip_0
- added link /human/left_hip_1
- added link /human/left_knee; visual cylinder length=0.370455770871 radius=0.025
- added link /human/left_leg_mount
- added link /human/left_shoulder; visual cylinder length=0.267443515341 radius=0.05
- added link /human/left_shoulder_0
- added link /human/left_shoulder_1
- added link /human/left_wrist; visual box size=0.1 0.05 .005
- added link /human/left_wrist_0
- added link /human/neck; visual cylinder length=0.26517305873 radius=0.04
- added link /human/neck_0
- added link /human/neck_1
- added link /human/right_ankle; visual box size=0.1 0.05 .005
- added link /human/right_ankle_0
- added link /human/right_arm_mount
- added link /human/right_elbow; visual cylinder length=0.226603262858 radius=0.025
- added link /human/right_elbow_0
- added link /human/right_foot
- added link /human/right_hand
- added link /human/right_hip; visual cylinder length=0.366580233013 radius=0.05
- added link /human/right_hip_0
- added link /human/right_hip_1
- added link /human/right_knee; visual cylinder length=0.370455770871 radius=0.025
- added link /human/right_leg_mount
- added link /human/right_shoulder; visual cylinder length=0.267443515341 radius=0.05
- added link /human/right_shoulder_0
- added link /human/right_shoulder_1
- added link /human/right_wrist; visual box size=0.1 0.05 .005
- added link /human/right_wrist_0
- added link /human/shoulder_center; visual cylinder length=0.0767374953016 radius=0.154143152453
- added link /human/spine; visual cylinder length=0.248644517245 radius=0.134143152453
- added link /human/spine_0; visual cylinder length=0.0666488013161 radius=0.114143152453
- added link /human/spine_1
- added link /human/spine_2
Joints:
- joint head: child head -> /human/head; origin xyz=0 0 0.194702136255 rpy=0 0 0 -> xyz=0 0 0.26517305873 rpy=0 0 0; parent neck -> /human/neck
- joint hip: child spine_0 -> /human/spine_0; parent base -> /human/base
- joint left_ankle_0: child left_ankle_0 -> /human/left_ankle_0; origin xyz=0.377295708046 0 0 rpy=-1.57079632679 0 1.57079632679 -> xyz=0.370455770871 0 0 rpy=-1.57079632679 0 1.57079632679; parent left_knee -> /human/left_knee
- joint left_ankle_1: child left_ankle -> /human/left_ankle; parent left_ankle_0 -> /human/left_ankle_0
- joint left_arm_mount: child left_arm_mount -> /human/left_arm_mount; origin xyz=0 0.19918889412 0.00217313207535 rpy=0 0 1.57079632679 -> xyz=0 0.154143152453 -0.0409013841447 rpy=0 0 1.57079632679; parent shoulder_center -> /human/shoulder_center
- joint left_elbow_0: child left_elbow_0 -> /human/left_elbow_0; origin xyz=0.298109797064 0 0 rpy=0 0 0 -> xyz=0.267443515341 0 0 rpy=0 0 0; parent left_shoulder -> /human/left_shoulder
- joint left_elbow_1: child left_elbow -> /human/left_elbow; parent left_elbow_0 -> /human/left_elbow_0
- joint left_foot: child left_foot -> /human/left_foot; parent left_ankle -> /human/left_ankle
- joint left_hand: child left_hand -> /human/left_hand; parent left_wrist -> /human/left_wrist
- joint left_hip_0: child left_hip_0 -> /human/left_hip_0; parent left_leg_mount -> /human/left_leg_mount
- joint left_hip_1: child left_hip_1 -> /human/left_hip_1; parent left_hip_0 -> /human/left_hip_0
- joint left_hip_2: child left_hip -> /human/left_hip; parent left_hip_1 -> /human/left_hip_1
- joint left_hip_leg_mount: child left_leg_mount -> /human/left_leg_mount; origin xyz=0 0.0823932168285 -0.0855449172121 rpy=0 1.57079632679 0 -> xyz=0 0.0693858304629 -0.106054276781 rpy=0 1.57079632679 0; parent base -> /human/base
- joint left_knee: child left_knee -> /human/left_knee; origin xyz=0.599774544438 0 0 rpy=1.57079632679 0 0 -> xyz=0.366580233013 0 0 rpy=1.57079632679 0 0; parent left_hip -> /human/left_hip
- joint left_shoulder_0: child left_shoulder_0 -> /human/left_shoulder_0; parent left_arm_mount -> /human/left_arm_mount
- joint left_shoulder_1: child left_shoulder_1 -> /human/left_shoulder_1; parent left_shoulder_0 -> /human/left_shoulder_0
- joint left_shoulder_2: child left_shoulder -> /human/left_shoulder; parent left_shoulder_1 -> /human/left_shoulder_1
- joint left_wrist_0: child left_wrist_0 -> /human/left_wrist_0; origin xyz=0.241500492953 0 0 rpy=0 0 0 -> xyz=0.226603262858 0 0 rpy=0 0 0; parent left_elbow -> /human/left_elbow
- joint left_wrist_1: child left_wrist -> /human/left_wrist; parent left_wrist_0 -> /human/left_wrist_0
- joint neck_0: child neck_0 -> /human/neck_0; origin xyz=0 0 0.105622495203 rpy=0 0 0 -> xyz=0 0 0.0767374953016 rpy=0 0 0; parent shoulder_center -> /human/shoulder_center
- joint neck_1: child neck_1 -> /human/neck_1; parent neck_0 -> /human/neck_0
- joint neck_2: child neck -> /human/neck; parent neck_1 -> /human/neck_1
- joint right_ankle_0: child right_ankle_0 -> /human/right_ankle_0; origin xyz=0.377295708046 0 0 rpy=-1.57079632679 0 1.57079632679 -> xyz=0.370455770871 0 0 rpy=-1.57079632679 0 1.57079632679; parent right_knee -> /human/right_knee
- joint right_ankle_1: child right_ankle -> /human/right_ankle; parent right_ankle_0 -> /human/right_ankle_0
- joint right_arm_mount: child right_arm_mount -> /human/right_arm_mount; origin xyz=0 -0.19918889412 0.00217313207535 rpy=0 0 -1.57079632679 -> xyz=0 -0.154143152453 -0.0409013841447 rpy=0 0 -1.57079632679; parent shoulder_center -> /human/shoulder_center
- joint right_elbow_0: child right_elbow_0 -> /human/right_elbow_0; origin xyz=0.298109797064 0 0 rpy=0 0 0 -> xyz=0.267443515341 0 0 rpy=0 0 0; parent right_shoulder -> /human/right_shoulder
- joint right_elbow_1: child right_elbow -> /human/right_elbow; parent right_elbow_0 -> /human/right_elbow_0
- joint right_foot: child right_foot -> /human/right_foot; parent right_ankle -> /human/right_ankle
- joint right_hand: child right_hand -> /human/right_hand; parent right_wrist -> /human/right_wrist
- joint right_hip_0: child right_hip_0 -> /human/right_hip_0; parent right_leg_mount -> /human/right_leg_mount
- joint right_hip_1: child right_hip_1 -> /human/right_hip_1; parent right_hip_0 -> /human/right_hip_0
- joint right_hip_2: child right_hip -> /human/right_hip; parent right_hip_1 -> /human/right_hip_1
- joint right_hip_leg_mount: child right_leg_mount -> /human/right_leg_mount; origin xyz=0 -0.0823932168285 -0.0855449172121 rpy=0 1.57079632679 0 -> xyz=0 -0.0693858304629 -0.106054276781 rpy=0 1.57079632679 0; parent base -> /human/base
- joint right_knee: child right_knee -> /human/right_knee; origin xyz=0.599774544438 0 0 rpy=1.57079632679 0 0 -> xyz=0.366580233013 0 0 rpy=1.57079632679 0 0; parent right_hip -> /human/right_hip
- joint right_shoulder_0: child right_shoulder_0 -> /human/right_shoulder_0; parent right_arm_mount -> /human/right_arm_mount
- joint right_shoulder_1: child right_shoulder_1 -> /human/right_shoulder_1; parent right_shoulder_0 -> /human/right_shoulder_0
- joint right_shoulder_2: child right_shoulder -> /human/right_shoulder; parent right_shoulder_1 -> /human/right_shoulder_1
- joint right_wrist_0: child right_wrist_0 -> /human/right_wrist_0; origin xyz=0.241500492953 0 0 rpy=0 0 0 -> xyz=0.226603262858 0 0 rpy=0 0 0; parent right_elbow -> /human/right_elbow
- joint right_wrist_1: child right_wrist -> /human/right_wrist; parent right_wrist_0 -> /human/right_wrist_0
- joint shoulder_center: child shoulder_center -> /human/shoulder_center; origin xyz=0 0 0.249607579586 rpy=0 0 0 -> xyz=0 0 0.248644517245 rpy=0 0 0; parent spine -> /human/spine
- joint spine_0: child spine_1 -> /human/spine_1; origin xyz=0 0 0.0838337572759 rpy=0 0 0 -> xyz=0 0 0.0666488013161 rpy=0 0 0; parent spine_0 -> /human/spine_0
- joint spine_1: child spine_2 -> /human/spine_2; parent spine_1 -> /human/spine_1
- joint spine_2: child spine -> /human/spine; parent spine_2 -> /human/spine_2

File: urdf/xacro/human_arm.urdf.xacro (robot description, xacro)
@@ -3,8 +3,8 @@
 <xacro:include filename="props_global.urdf.xacro" />
 <xacro:macro name="human_arm" params="side reflect boolside">
-    <link name="${side}_arm_mount"/>
-    <link name="${side}_shoulder_0"/>
-    <link name="${side}_shoulder_1"/>
-    <link name="${side}_shoulder">
+    <link name="${prefix}/${side}_arm_mount"/>
+    <link name="${prefix}/${side}_shoulder_0"/>
+    <link name="${prefix}/${side}_shoulder_1"/>
+    <link name="${prefix}/${side}_shoulder">
       <visual>
         <origin xyz="${upper_arm_length/2} 0 0" rpy="0 ${PI_DIV_2} 0" />
@@ -14,6 +14,6 @@
       </visual>
     </link>
-    <link name="${side}_elbow_0"/>
-    <link name="${side}_elbow">
+    <link name="${prefix}/${side}_elbow_0"/>
+    <link name="${prefix}/${side}_elbow">
       <visual>
         <origin xyz="${forearm_length/2} 0 0" rpy="0 ${PI_DIV_2} 0" />
@@ -23,6 +23,6 @@
       </visual>
     </link>
-    <link name="${side}_wrist_0"/>
-    <link name="${side}_wrist">
+    <link name="${prefix}/${side}_wrist_0"/>
+    <link name="${prefix}/${side}_wrist">
       <visual>
         <origin xyz="${hand_length/2} 0 0" rpy="0 0 0" />
@@ -32,10 +32,10 @@
       </visual>
     </link>
-    <link name="${side}_hand"/>
+    <link name="${prefix}/${side}_hand"/>
     <!-- Joints -->
     <joint name="${side}_arm_mount" type="fixed">
       <origin xyz="0 ${reflect*shoulder_offset_width} ${shoulder_offset_height}" rpy="0 0 ${reflect*PI_DIV_2}" />
-      <parent link="shoulder_center" />
-      <child link="${side}_arm_mount" />
+      <parent link="${prefix}/shoulder_center" />
+      <child link="${prefix}/${side}_arm_mount" />
     </joint>
     <!-- SHOULDER : spherical -->
@@ -43,6 +43,6 @@
           <origin xyz="0 0 0" rpy="0 0 0" />
           <axis xyz="0 1 0" />
-          <parent link="${side}_arm_mount" />
-          <child link="${side}_shoulder_0" />
+          <parent link="${prefix}/${side}_arm_mount" />
+          <child link="${prefix}/${side}_shoulder_0" />
           <limit lower="${-PI_DIV_2}" upper="${PI_DIV_2}" effort="${max_effort}" velocity="${max_velocity}"  />
         </joint>
@@ -51,6 +51,6 @@
             <origin xyz="0 0 0" rpy="0 0 0" />
             <axis xyz="0 0 1" />
-            <parent link="left_shoulder_0" />
-            <child link="left_shoulder_1" />
+            <parent link="${prefix}/left_shoulder_0" />
+            <child link="${prefix}/left_shoulder_1" />
             <limit lower="${-TPI_DIV_4}" upper="${PI_DIV_2}" effort="${max_effort}" velocity="${max_velocity}"  />
           </joint>
@@ -60,6 +60,6 @@
             <origin xyz="0 0 0" rpy="0 0 0" />
             <axis xyz="0 0 1" />
-            <parent link="right_shoulder_0" />
-            <child link="right_shoulder_1" />
+            <parent link="${prefix}/right_shoulder_0" />
+            <child link="${prefix}/right_shoulder_1" />
             <limit lower="${-PI_DIV_2}" upper="${TPI_DIV_4}" effort="${max_effort}" velocity="${max_velocity}"  />
           </joint>
@@ -68,6 +68,6 @@
           <origin xyz="0 0 0" rpy="0 0 0" />
           <axis xyz="1 0 0" />
-          <parent link="${side}_shoulder_1" />
-          <child link="${side}_shoulder" />
+          <parent link="${prefix}/${side}_shoulder_1" />
+          <child link="${prefix}/${side}_shoulder" />
           <limit lower="${-PI_DIV_2}" upper="${PI_DIV_2}" effort="${max_effort}" velocity="${max_velocity}"  />
         </joint>
@@ -77,6 +77,6 @@
         <origin xyz="${upper_arm_length} 0 0" rpy="0 0 0" />
         <axis xyz="0 0 1" />
-        <parent link="left_shoulder" />
-        <child link="left_elbow_0" />
+        <parent link="${prefix}/left_shoulder" />
+        <child link="${prefix}/left_elbow_0" />
         <limit lower="${-PI}" upper="0.0" effort="${max_effort}" velocity="${max_velocity}"  />
       </joint>
@@ -84,6 +84,6 @@
         <origin xyz="0 0 0" rpy="0 0 0" />
         <axis xyz="1 0 0" />
-        <parent link="left_elbow_0" />
-        <child link="left_elbow" />
+        <parent link="${prefix}/left_elbow_0" />
+        <child link="${prefix}/left_elbow" />
         <limit lower="${-PI}" upper="0.0" effort="${max_effort}" velocity="${max_velocity}"  />
       </joint>
@@ -93,6 +93,6 @@
         <origin xyz="${upper_arm_length} 0 0" rpy="0 0 0" />
         <axis xyz="0 0 1" />
-        <parent link="right_shoulder" />
-        <child link="right_elbow_0" />
+        <parent link="${prefix}/right_shoulder" />
+        <child link="${prefix}/right_elbow_0" />
         <limit lower="0.0" upper="${PI}" effort="${max_effort}" velocity="${max_velocity}"  />
       </joint>
@@ -100,6 +100,6 @@
         <origin xyz="0 0 0" rpy="0 0 0" />
         <axis xyz="1 0 0" />
-        <parent link="right_elbow_0" />
-        <child link="right_elbow" />
+        <parent link="${prefix}/right_elbow_0" />
+        <child link="${prefix}/right_elbow" />
         <limit lower="0.0" upper="${PI}" effort="${max_effort}" velocity="${max_velocity}"  />
       </joint>
@@ -108,6 +108,6 @@
       <origin xyz="${forearm_length} 0 0" rpy="0 0 0" />
       <axis xyz="0 0 1" />
-      <parent link="${side}_elbow" />
-      <child link="${side}_wrist_0" />
+      <parent link="${prefix}/${side}_elbow" />
+      <child link="${prefix}/${side}_wrist_0" />
       <limit lower="${-PI_DIV_4}" upper="${PI_DIV_4}" effort="${max_effort}" velocity="${max_velocity}"  />
     </joint>
@@ -115,12 +115,12 @@
       <origin xyz="0 0 0" rpy="0 0 0" />
       <axis xyz="0 1 0" />
-      <parent link="${side}_wrist_0" />
-      <child link="${side}_wrist" />
+      <parent link="${prefix}/${side}_wrist_0" />
+      <child link="${prefix}/${side}_wrist" />
       <limit lower="${-PI_DIV_2}" upper="${PI_DIV_2}" effort="${max_effort}" velocity="${max_velocity}"  />
     </joint>
     <joint name="${side}_hand" type="fixed">
       <origin xyz="${hand_length} 0 0" rpy="0 0 0" />
-      <parent link="${side}_wrist" />
-      <child link="${side}_hand" />
+      <parent link="${prefix}/${side}_wrist" />
+      <child link="${prefix}/${side}_hand" />
     </joint>
 </xacro:macro>

File: urdf/xacro/human_body.urdf.xacro (robot description, xacro)
@@ -3,5 +3,5 @@
 <xacro:include filename="props_global.urdf.xacro" />
 <xacro:macro name="human_body">
-	  <link name="base">
+	  <link name="${prefix}/base">
       <visual>
         <origin xyz="0 0 ${-hip_offset_height/2}" rpy="0 0 0" />
@@ -11,5 +11,5 @@
       </visual>
     </link>
-    <link name="spine_0">
+    <link name="${prefix}/spine_0">
       <visual>
         <origin xyz="0 0 ${spine_down_length/2}" rpy="0 0 0" />
@@ -19,7 +19,7 @@
       </visual>
     </link>
-    <link name="spine_1"/>
-    <link name="spine_2"/>
-    <link name="spine">
+    <link name="${prefix}/spine_1"/>
+    <link name="${prefix}/spine_2"/>
+    <link name="${prefix}/spine">
       <visual>
         <origin xyz="0 0 ${spine_up_length/2}" rpy="0 0 0" />
@@ -29,5 +29,5 @@
       </visual>
     </link>
-    <link name="shoulder_center">
+    <link name="${prefix}/shoulder_center">
       <visual>
         <origin xyz="0 0 ${torso_length/2}" rpy="0 0 0" />
@@ -37,7 +37,7 @@
       </visual>
     </link>
-    <link name="neck_0"/>
-    <link name="neck_1"/>
-    <link name="neck">
+    <link name="${prefix}/neck_0"/>
+    <link name="${prefix}/neck_1"/>
+    <link name="${prefix}/neck">
       <visual>
         <origin xyz="0 0 ${neck_length/2}" rpy="0 0 0" />
@@ -47,5 +47,5 @@
       </visual>
     </link>
-    <link name="head">
+    <link name="${prefix}/head">
       <visual>
         <origin xyz="0 0 0" rpy="0 0 0" />
@@ -57,6 +57,6 @@
     <joint name="hip" type="fixed">
       <origin xyz="0 0 0" rpy="0 0 0" />
-      <parent link="base" />
-      <child link="spine_0" />
+      <parent link="${prefix}/base" />
+      <child link="${prefix}/spine_0" />
     </joint>
     <!-- SPINE : spherical -->
@@ -64,6 +64,6 @@
       <origin xyz="0 0 ${spine_down_length}" rpy="0 0 0" />
       <axis xyz="1 0 0" />
-      <parent link="spine_0" />
-      <child link="spine_1" />
+      <parent link="${prefix}/spine_0" />
+      <child link="${prefix}/spine_1" />
       <limit lower="${-PI_DIV_2}" upper="${PI_DIV_2}" effort="${max_effort}" velocity="${max_velocity}" />
     </joint>
@@ -71,6 +71,6 @@
       <origin xyz="0 0 0" rpy="0 0 0" />
       <axis xyz="0 1 0" />
-      <parent link="spine_1" />
-      <child link="spine_2" />
+      <parent link="${prefix}/spine_1" />
+      <child link="${prefix}/spine_2" />
       <limit lower="${-PI_DIV_2}" upper="${PI_DIV_2}" effort="${max_effort}" velocity="${max_velocity}" />
     </joint>
@@ -78,12 +78,12 @@
       <origin xyz="0 0 0" rpy="0 0 0" />
       <axis xyz="0 0 1" />
-      <parent link="spine_2" />
-      <child link="spine" />
+      <parent link="${prefix}/spine_2" />
+      <child link="${prefix}/spine" />
       <limit lower="${-PI_DIV_2}" upper="${PI_DIV_2}" effort="${max_effort}" velocity="${max_velocity}" />
     </joint>
     <joint name="shoulder_center" type="fixed">
       <origin xyz="0 0 ${spine_up_length}" rpy="0 0 0" />
-      <parent link="spine" />
-      <child link="shoulder_center" />
+      <parent link="${prefix}/spine" />
+      <child link="${prefix}/shoulder_center" />
     </joint>
     <!-- NECK : spherical -->
@@ -91,6 +91,6 @@
           <origin xyz="0 0 ${torso_length}" rpy="0 0 0" />
           <axis xyz="1 0 0" />
-          <parent link="shoulder_center" />
-          <child link="neck_0" />
+          <parent link="${prefix}/shoulder_center" />
+          <child link="${prefix}/neck_0" />
           <limit lower="${-PI_DIV_2}" upper="${PI_DIV_2}" effort="${max_effort}" velocity="${max_velocity}"  />
         </joint>
@@ -98,6 +98,6 @@
           <origin xyz="0 0 0" rpy="0 0 0" />
           <axis xyz="0 1 0" />
-          <parent link="neck_0" />
-          <child link="neck_1" />
+          <parent link="${prefix}/neck_0" />
+          <child link="${prefix}/neck_1" />
           <limit lower="${-PI_DIV_2}" upper="${PI_DIV_2}" effort="${max_effort}" velocity="${max_velocity}"  />
         </joint>
@@ -105,6 +105,6 @@
           <origin xyz="0 0 0" rpy="0 0 0" />
           <axis xyz="0 0 1" />
-          <parent link="neck_1" />
-          <child link="neck" />
+          <parent link="${prefix}/neck_1" />
+          <child link="${prefix}/neck" />
           <limit lower="${-PI_DIV_2}" upper="${PI_DIV_2}" effort="${max_effort}" velocity="${max_velocity}" />
         </joint>
@@ -112,6 +112,6 @@
     <joint name="head" type="fixed">
       <origin xyz="0 0 ${neck_length}" rpy="0 0 0" />
-      <parent link="neck" />
-      <child link="head" />
+      <parent link="${prefix}/neck" />
+      <child link="${prefix}/head" />
     </joint>
 </xacro:macro>
