Commit message: Add a prefix to each link of the URDF to avoid conflicts with Baxter

File: urdf/xacro/human_leg.urdf.xacro (robot description, xacro)
@@ -3,8 +3,8 @@
 <xacro:include filename="props_global.urdf.xacro" />
 <xacro:macro name="human_leg" params="side reflect">
-    <link name="${side}_leg_mount"/>
-    <link name="${side}_hip_0"/>
-    <link name="${side}_hip_1"/>
-    <link name="${side}_hip">
+    <link name="${prefix}/${side}_leg_mount"/>
+    <link name="${prefix}/${side}_hip_0"/>
+    <link name="${prefix}/${side}_hip_1"/>
+    <link name="${prefix}/${side}_hip">
       <visual>
         <origin xyz="${thigh_length/2} 0 0" rpy="0 ${PI_DIV_2} 0" />
@@ -14,5 +14,5 @@
       </visual>
     </link>
-    <link name="${side}_knee">
+    <link name="${prefix}/${side}_knee">
       <visual>
         <origin xyz="${shin_length/2} 0 0" rpy="0 ${PI_DIV_2} 0" />
@@ -22,6 +22,6 @@
       </visual>
     </link>
-    <link name="${side}_ankle_0"/>
-    <link name="${side}_ankle">
+    <link name="${prefix}/${side}_ankle_0"/>
+    <link name="${prefix}/${side}_ankle">
       <visual>
         <origin xyz="${foot_length/2} 0 0" rpy="0 0 0" />
@@ -31,10 +31,10 @@
       </visual>
     </link>
-    <link name="${side}_foot"/>
+    <link name="${prefix}/${side}_foot"/>
     <!-- Joints -->
     <joint name="${side}_hip_leg_mount" type="fixed">
       <origin xyz="0 ${reflect*hip_offset_width} ${-hip_offset_height}" rpy="0 ${PI_DIV_2} 0" />
-      <parent link="base" />
-      <child link="${side}_leg_mount" />
+      <parent link="${prefix}/base" />
+      <child link="${prefix}/${side}_leg_mount" />
     </joint>
     <!-- hip : spherical -->
@@ -42,6 +42,6 @@
           <origin xyz="0 0 0" rpy="0 0 0" />
           <axis xyz="0 0 1" />
-          <parent link="${side}_leg_mount" />
-          <child link="${side}_hip_0" />
+          <parent link="${prefix}/${side}_leg_mount" />
+          <child link="${prefix}/${side}_hip_0" />
           <limit lower="${-PI_DIV_2}" upper="${PI_DIV_2}" effort="${max_effort}" velocity="${max_velocity}"  />
         </joint>
@@ -49,6 +49,6 @@
           <origin xyz="0 0 0" rpy="0 0 0" />
           <axis xyz="0 1 0" />
-          <parent link="${side}_hip_0" />
-          <child link="${side}_hip_1" />
+          <parent link="${prefix}/${side}_hip_0" />
+          <child link="${prefix}/${side}_hip_1" />
           <limit lower="${-PI_DIV_2}" upper="${PI_DIV_2}" effort="${max_effort}" velocity="${max_velocity}"  />
         </joint>
@@ -56,6 +56,6 @@
           <origin xyz="0 0 0" rpy="0 0 0" />
           <axis xyz="1 0 0" />
-          <parent link="${side}_hip_1" />
-          <child link="${side}_hip" />
+          <parent link="${prefix}/${side}_hip_1" />
+          <child link="${prefix}/${side}_hip" />
           <limit lower="${-PI_DIV_2}" upper="${PI_DIV_2}" effort="${max_effort}" velocity="${max_velocity}"  />
         </joint>
@@ -64,6 +64,6 @@
       <origin xyz="${thigh_length} 0 0" rpy="${PI_DIV_2} 0 0" />
       <axis xyz="0 0 1" />
-      <parent link="${side}_hip" />
-      <child link="${side}_knee" />
+      <parent link="${prefix}/${side}_hip" />
+      <child link="${prefix}/${side}_knee" />
       <limit lower="${-PI}" upper="0.1" effort="${max_effort}" velocity="${max_velocity}"  />
     </joint>
@@ -72,6 +72,6 @@
           <origin xyz="${shin_length} 0 0" rpy="${-PI_DIV_2} 0 ${PI_DIV_2}" />
           <axis xyz="0 0 1" />
-          <parent link="${side}_knee" />
-          <child link="${side}_ankle_0" />
+          <parent link="${prefix}/${side}_knee" />
+          <child link="${prefix}/${side}_ankle_0" />
           <limit lower="${-PI_DIV_2}" upper="${PI_DIV_2}" effort="${max_effort}" velocity="${max_velocity}"  />
         </joint>
@@ -79,6 +79,6 @@
           <origin xyz="0 0 0" rpy="0 0 0" />
           <axis xyz="0 1 0" />
-          <parent link="${side}_ankle_0" />
-          <child link="${side}_ankle" />
+          <parent link="${prefix}/${side}_ankle_0" />
+          <child link="${prefix}/${side}_ankle" />
           <limit lower="${-PI_DIV_2}" upper="${PI_DIV_2}" effort="${max_effort}" velocity="${max_velocity}" />
         </joint>
@@ -86,6 +86,6 @@
     <joint name="${side}_foot" type="fixed">
       <origin xyz="${foot_length} 0 0" rpy="0 0 0" />
-      <parent link="${side}_ankle" />
-      <child link="${side}_foot" />
+      <parent link="${prefix}/${side}_ankle" />
+      <child link="${prefix}/${side}_foot" />
     </joint>
 </xacro:macro>

File: urdf/xacro/props_global.urdf.xacro (robot description, xacro)
@@ -1,4 +1,5 @@
 <?xml version="1.0"?>
 <robot xmlns:xacro="http://playerstage.sourceforge.net/gazebo/xmlschema/#interface" name="human_model" >
+  <xacro:property name="prefix" value="/human" />
   <xacro:property name="PI" value="3.14159265359" />
   <xacro:property name="PI_DIV_2" value="1.5707963267948966" />

Commit message: Replace prefix /human by human

File: urdf/human.urdf (robot description, URDF)
Before this commit: robot human_model, 44 links, 43 joints
Links:
- removed link /human/base
- removed link /human/head
- removed link /human/left_ankle
- removed link /human/left_ankle_0
- removed link /human/left_arm_mount
- removed link /human/left_elbow
- removed link /human/left_elbow_0
- removed link /human/left_foot
- removed link /human/left_hand
- removed link /human/left_hip
- removed link /human/left_hip_0
- removed link /human/left_hip_1
- removed link /human/left_knee
- removed link /human/left_leg_mount
- removed link /human/left_shoulder
- removed link /human/left_shoulder_0
- removed link /human/left_shoulder_1
- removed link /human/left_wrist
- removed link /human/left_wrist_0
- removed link /human/neck
- removed link /human/neck_0
- removed link /human/neck_1
- removed link /human/right_ankle
- removed link /human/right_ankle_0
- removed link /human/right_arm_mount
- removed link /human/right_elbow
- removed link /human/right_elbow_0
- removed link /human/right_foot
- removed link /human/right_hand
- removed link /human/right_hip
- removed link /human/right_hip_0
- removed link /human/right_hip_1
- removed link /human/right_knee
- removed link /human/right_leg_mount
- removed link /human/right_shoulder
- removed link /human/right_shoulder_0
- removed link /human/right_shoulder_1
- removed link /human/right_wrist
- removed link /human/right_wrist_0
- removed link /human/shoulder_center
- removed link /human/spine
- removed link /human/spine_0
- removed link /human/spine_1
- removed link /human/spine_2
- added link human/base; visual cylinder length=-0.069200086074 radius=0.123726284724
- added link human/head; visual sphere radius=0.1
- added link human/left_ankle; visual box size=0.1 0.05 .005
- added link human/left_ankle_0
- added link human/left_arm_mount
- added link human/left_elbow; visual cylinder length=0.29962489513 radius=0.025
- added link human/left_elbow_0
- added link human/left_foot
- added link human/left_hand
- added link human/left_hip; visual cylinder length=0.449062644944 radius=0.05
- added link human/left_hip_0
- added link human/left_hip_1
- added link human/left_knee; visual cylinder length=0.289568127664 radius=0.025
- added link human/left_leg_mount
- added link human/left_shoulder; visual cylinder length=0.310233775399 radius=0.05
- added link human/left_shoulder_0
- added link human/left_shoulder_1
- added link human/left_wrist; visual box size=0.1 0.05 .005
- added link human/left_wrist_0
- added link human/neck; visual cylinder length=0.176495586912 radius=0.04
- added link human/neck_0
- added link human/neck_1
- added link human/right_ankle; visual box size=0.1 0.05 .005
- added link human/right_ankle_0
- added link human/right_arm_mount
- added link human/right_elbow; visual cylinder length=0.29962489513 radius=0.025
- added link human/right_elbow_0
- added link human/right_foot
- added link human/right_hand
- added link human/right_hip; visual cylinder length=0.449062644944 radius=0.05
- added link human/right_hip_0
- added link human/right_hip_1
- added link human/right_knee; visual cylinder length=0.289568127664 radius=0.025
- added link human/right_leg_mount
- added link human/right_shoulder; visual cylinder length=0.310233775399 radius=0.05
- added link human/right_shoulder_0
- added link human/right_shoulder_1
- added link human/right_wrist; visual box size=0.1 0.05 .005
- added link human/right_wrist_0
- added link human/shoulder_center; visual cylinder length=0.121005899273 radius=0.162221019628
- added link human/spine; visual cylinder length=0.241077936334 radius=0.142221019628
- added link human/spine_0; visual cylinder length=0.0838556756279 radius=0.122221019628
- added link human/spine_1
- added link human/spine_2
Joints:
- joint head: child /human/head -> human/head; origin xyz=0 0 0.26517305873 rpy=0 0 0 -> xyz=0 0 0.176495586912 rpy=0 0 0; parent /human/neck -> human/neck
- joint hip: child /human/spine_0 -> human/spine_0; parent /human/base -> human/base
- joint left_ankle_0: child /human/left_ankle_0 -> human/left_ankle_0; origin xyz=0.370455770871 0 0 rpy=-1.57079632679 0 1.57079632679 -> xyz=0.289568127664 0 0 rpy=-1.57079632679 0 1.57079632679; parent /human/left_knee -> human/left_knee
- joint left_ankle_1: child /human/left_ankle -> human/left_ankle; parent /human/left_ankle_0 -> human/left_ankle_0
- joint left_arm_mount: child /human/left_arm_mount -> human/left_arm_mount; origin xyz=0 0.154143152453 -0.0409013841447 rpy=0 0 1.57079632679 -> xyz=0 0.162221019628 0.000148014454256 rpy=0 0 1.57079632679; parent /human/shoulder_center -> human/shoulder_center
- joint left_elbow_0: child /human/left_elbow_0 -> human/left_elbow_0; origin xyz=0.267443515341 0 0 rpy=0 0 0 -> xyz=0.310233775399 0 0 rpy=0 0 0; parent /human/left_shoulder -> human/left_shoulder
- joint left_elbow_1: child /human/left_elbow -> human/left_elbow; parent /human/left_elbow_0 -> human/left_elbow_0
- joint left_foot: child /human/left_foot -> human/left_foot; parent /human/left_ankle -> human/left_ankle
- joint left_hand: child /human/left_hand -> human/left_hand; parent /human/left_wrist -> human/left_wrist
- joint left_hip_0: child /human/left_hip_0 -> human/left_hip_0; parent /human/left_leg_mount -> human/left_leg_mount
- joint left_hip_1: child /human/left_hip_1 -> human/left_hip_1; parent /human/left_hip_0 -> human/left_hip_0
- joint left_hip_2: child /human/left_hip -> human/left_hip; parent /human/left_hip_1 -> human/left_hip_1
- joint left_hip_leg_mount: child /human/left_leg_mount -> human/left_leg_mount; origin xyz=0 0.0693858304629 -0.106054276781 rpy=0 1.57079632679 0 -> xyz=0 0.0737262847244 -0.069200086074 rpy=0 1.57079632679 0; parent /human/base -> human/base
- joint left_knee: child /human/left_knee -> human/left_knee; origin xyz=0.366580233013 0 0 rpy=1.57079632679 0 0 -> xyz=0.449062644944 0 0 rpy=1.57079632679 0 0; parent /human/left_hip -> human/left_hip
- joint left_shoulder_0: child /human/left_shoulder_0 -> human/left_shoulder_0; parent /human/left_arm_mount -> human/left_arm_mount
- joint left_shoulder_1: child /human/left_shoulder_1 -> human/left_shoulder_1; parent /human/left_shoulder_0 -> human/left_shoulder_0
- joint left_shoulder_2: child /human/left_shoulder -> human/left_shoulder; parent /human/left_shoulder_1 -> human/left_shoulder_1
- joint left_wrist_0: child /human/left_wrist_0 -> human/left_wrist_0; origin xyz=0.226603262858 0 0 rpy=0 0 0 -> xyz=0.29962489513 0 0 rpy=0 0 0; parent /human/left_elbow -> human/left_elbow
- joint left_wrist_1: child /human/left_wrist -> human/left_wrist; parent /human/left_wrist_0 -> human/left_wrist_0
- joint neck_0: child /human/neck_0 -> human/neck_0; origin xyz=0 0 0.0767374953016 rpy=0 0 0 -> xyz=0 0 0.121005899273 rpy=0 0 0; parent /human/shoulder_center -> human/shoulder_center
- joint neck_1: child /human/neck_1 -> human/neck_1; parent /human/neck_0 -> human/neck_0
- joint neck_2: child /human/neck -> human/neck; parent /human/neck_1 -> human/neck_1
- joint right_ankle_0: child /human/right_ankle_0 -> human/right_ankle_0; origin xyz=0.370455770871 0 0 rpy=-1.57079632679 0 1.57079632679 -> xyz=0.289568127664 0 0 rpy=-1.57079632679 0 1.57079632679; parent /human/right_knee -> human/right_knee
- joint right_ankle_1: child /human/right_ankle -> human/right_ankle; parent /human/right_ankle_0 -> human/right_ankle_0
- joint right_arm_mount: child /human/right_arm_mount -> human/right_arm_mount; origin xyz=0 -0.154143152453 -0.0409013841447 rpy=0 0 -1.57079632679 -> xyz=0 -0.162221019628 0.000148014454256 rpy=0 0 -1.57079632679; parent /human/shoulder_center -> human/shoulder_center
- joint right_elbow_0: child /human/right_elbow_0 -> human/right_elbow_0; origin xyz=0.267443515341 0 0 rpy=0 0 0 -> xyz=0.310233775399 0 0 rpy=0 0 0; parent /human/right_shoulder -> human/right_shoulder
- joint right_elbow_1: child /human/right_elbow -> human/right_elbow; parent /human/right_elbow_0 -> human/right_elbow_0
- joint right_foot: child /human/right_foot -> human/right_foot; parent /human/right_ankle -> human/right_ankle
- joint right_hand: child /human/right_hand -> human/right_hand; parent /human/right_wrist -> human/right_wrist
- joint right_hip_0: child /human/right_hip_0 -> human/right_hip_0; parent /human/right_leg_mount -> human/right_leg_mount
- joint right_hip_1: child /human/right_hip_1 -> human/right_hip_1; parent /human/right_hip_0 -> human/right_hip_0
- joint right_hip_2: child /human/right_hip -> human/right_hip; parent /human/right_hip_1 -> human/right_hip_1
- joint right_hip_leg_mount: child /human/right_leg_mount -> human/right_leg_mount; origin xyz=0 -0.0693858304629 -0.106054276781 rpy=0 1.57079632679 0 -> xyz=0 -0.0737262847244 -0.069200086074 rpy=0 1.57079632679 0; parent /human/base -> human/base
- joint right_knee: child /human/right_knee -> human/right_knee; origin xyz=0.366580233013 0 0 rpy=1.57079632679 0 0 -> xyz=0.449062644944 0 0 rpy=1.57079632679 0 0; parent /human/right_hip -> human/right_hip
- joint right_shoulder_0: child /human/right_shoulder_0 -> human/right_shoulder_0; parent /human/right_arm_mount -> human/right_arm_mount
- joint right_shoulder_1: child /human/right_shoulder_1 -> human/right_shoulder_1; parent /human/right_shoulder_0 -> human/right_shoulder_0
- joint right_shoulder_2: child /human/right_shoulder -> human/right_shoulder; parent /human/right_shoulder_1 -> human/right_shoulder_1
- joint right_wrist_0: child /human/right_wrist_0 -> human/right_wrist_0; origin xyz=0.226603262858 0 0 rpy=0 0 0 -> xyz=0.29962489513 0 0 rpy=0 0 0; parent /human/right_elbow -> human/right_elbow
- joint right_wrist_1: child /human/right_wrist -> human/right_wrist; parent /human/right_wrist_0 -> human/right_wrist_0
- joint shoulder_center: child /human/shoulder_center -> human/shoulder_center; origin xyz=0 0 0.248644517245 rpy=0 0 0 -> xyz=0 0 0.241077936334 rpy=0 0 0; parent /human/spine -> human/spine
- joint spine_0: child /human/spine_1 -> human/spine_1; origin xyz=0 0 0.0666488013161 rpy=0 0 0 -> xyz=0 0 0.0838556756279 rpy=0 0 0; parent /human/spine_0 -> human/spine_0
- joint spine_1: child /human/spine_2 -> human/spine_2; parent /human/spine_1 -> human/spine_1
- joint spine_2: child /human/spine -> human/spine; parent /human/spine_2 -> human/spine_2

Commit message: Changes in URDF file
- joint elbow_1 changed to wrist_2: more anatomically correct
- joint knee changed to knee_0: consistency with other joint names

File: urdf/human.urdf (robot description, URDF)
Before this commit: robot human_model, 44 links, 43 joints
Links:
- removed link human/left_elbow_0
- removed link human/right_elbow_0
- added link human/left_wrist_1
- added link human/right_wrist_1
- link human/base: geometry visual cylinder length=-0.076637666482 radius=0.128063809513
- link human/left_elbow: geometry visual cylinder length=0.273206361701 radius=0.025
- link human/left_hip: geometry visual cylinder length=0.53151880807 radius=0.05
- link human/left_knee: geometry visual cylinder length=0.36903984413 radius=0.025
- link human/left_shoulder: geometry visual cylinder length=0.343212242182 radius=0.05
- link human/neck: geometry visual cylinder length=0.198713359681 radius=0.04
- link human/right_elbow: geometry visual cylinder length=0.273206361701 radius=0.025
- link human/right_hip: geometry visual cylinder length=0.53151880807 radius=0.05
- link human/right_knee: geometry visual cylinder length=0.36903984413 radius=0.025
- link human/right_shoulder: geometry visual cylinder length=0.343212242182 radius=0.05
- link human/shoulder_center: geometry visual cylinder length=0.126849441152 radius=0.173623764208
- link human/spine: geometry visual cylinder length=0.262448400938 radius=0.153623764208
- link human/spine_0: geometry visual cylinder length=0.0900777328402 radius=0.133623764208
Joints:
- removed joint left_elbow_1
- removed joint left_knee
- removed joint right_elbow_1
- removed joint right_knee
- added joint left_knee_0: type revolute, parent human/left_hip, child human/left_knee, origin xyz=0.53151880807 0 0 rpy=1.57079632679 0 0, axis 0 0 1, limit lower=-3.14159265359 upper=0.1 effort=1 velocity=1
- added joint left_wrist_2: type revolute, parent human/left_wrist_1, child human/left_wrist, origin xyz=0 0 0 rpy=0 0 0, axis 1 0 0, limit lower=-1.57079632679 upper=1.57079632679 effort=1 velocity=1
- added joint right_knee_0: type revolute, parent human/right_hip, child human/right_knee, origin xyz=0.53151880807 0 0 rpy=1.57079632679 0 0, axis 0 0 1, limit lower=-3.14159265359 upper=0.1 effort=1 velocity=1
- added joint right_wrist_2: type revolute, parent human/right_wrist_1, child human/right_wrist, origin xyz=0 0 0 rpy=0 0 0, axis 1 0 0, limit lower=-1.57079632679 upper=1.57079632679 effort=1 velocity=1
- joint head: origin xyz=0 0 0.176495586912 rpy=0 0 0 -> xyz=0 0 0.198713359681 rpy=0 0 0
- joint left_ankle_0: origin xyz=0.289568127664 0 0 rpy=-1.57079632679 0 1.57079632679 -> xyz=0.36903984413 0 0 rpy=-1.57079632679 0 1.57079632679
- joint left_arm_mount: origin xyz=0 0.162221019628 0.000148014454256 rpy=0 0 1.57079632679 -> xyz=0 0.173623764208 -0.00143826424372 rpy=0 0 1.57079632679
- joint left_elbow_0: child human/left_elbow_0 -> human/left_elbow; origin xyz=0.310233775399 0 0 rpy=0 0 0 -> xyz=0.343212242182 0 0 rpy=0 0 0
- joint left_hip_leg_mount: origin xyz=0 0.0737262847244 -0.069200086074 rpy=0 1.57079632679 0 -> xyz=0 0.0780638095132 -0.076637666482 rpy=0 1.57079632679 0
- joint left_wrist_0: origin xyz=0.29962489513 0 0 rpy=0 0 0 -> xyz=0.273206361701 0 0 rpy=0 0 0
- joint left_wrist_1: child human/left_wrist -> human/left_wrist_1
- joint neck_0: origin xyz=0 0 0.121005899273 rpy=0 0 0 -> xyz=0 0 0.126849441152 rpy=0 0 0
- joint right_ankle_0: origin xyz=0.289568127664 0 0 rpy=-1.57079632679 0 1.57079632679 -> xyz=0.36903984413 0 0 rpy=-1.57079632679 0 1.57079632679
- joint right_arm_mount: origin xyz=0 -0.162221019628 0.000148014454256 rpy=0 0 -1.57079632679 -> xyz=0 -0.173623764208 -0.00143826424372 rpy=0 0 -1.57079632679
- joint right_elbow_0: child human/right_elbow_0 -> human/right_elbow; origin xyz=0.310233775399 0 0 rpy=0 0 0 -> xyz=0.343212242182 0 0 rpy=0 0 0
- joint right_hip_leg_mount: origin xyz=0 -0.0737262847244 -0.069200086074 rpy=0 1.57079632679 0 -> xyz=0 -0.0780638095132 -0.076637666482 rpy=0 1.57079632679 0
- joint right_wrist_0: origin xyz=0.29962489513 0 0 rpy=0 0 0 -> xyz=0.273206361701 0 0 rpy=0 0 0
- joint right_wrist_1: child human/right_wrist -> human/right_wrist_1
- joint shoulder_center: origin xyz=0 0 0.241077936334 rpy=0 0 0 -> xyz=0 0 0.262448400938 rpy=0 0 0
- joint spine_0: origin xyz=0 0 0.0838556756279 rpy=0 0 0 -> xyz=0 0 0.0900777328402 rpy=0 0 0

File: urdf/xacro/human_arm.urdf.xacro (robot description, xacro)
@@ -14,5 +14,4 @@
       </visual>
     </link>
-    <link name="${prefix}/${side}_elbow_0"/>
     <link name="${prefix}/${side}_elbow">
       <visual>
@@ -24,4 +23,5 @@
     </link>
     <link name="${prefix}/${side}_wrist_0"/>
+    <link name="${prefix}/${side}_wrist_1"/>
     <link name="${prefix}/${side}_wrist">
       <visual>
@@ -78,11 +78,4 @@
         <axis xyz="0 0 1" />
         <parent link="${prefix}/left_shoulder" />
-        <child link="${prefix}/left_elbow_0" />
-        <limit lower="${-PI}" upper="0.0" effort="${max_effort}" velocity="${max_velocity}"  />
-      </joint>
-      <joint name="left_elbow_1" type="revolute">
-        <origin xyz="0 0 0" rpy="0 0 0" />
-        <axis xyz="1 0 0" />
-        <parent link="${prefix}/left_elbow_0" />
         <child link="${prefix}/left_elbow" />
         <limit lower="${-PI}" upper="0.0" effort="${max_effort}" velocity="${max_velocity}"  />
@@ -94,11 +87,4 @@
         <axis xyz="0 0 1" />
         <parent link="${prefix}/right_shoulder" />
-        <child link="${prefix}/right_elbow_0" />
-        <limit lower="0.0" upper="${PI}" effort="${max_effort}" velocity="${max_velocity}"  />
-      </joint>
-      <joint name="right_elbow_1" type="revolute">
-        <origin xyz="0 0 0" rpy="0 0 0" />
-        <axis xyz="1 0 0" />
-        <parent link="${prefix}/right_elbow_0" />
         <child link="${prefix}/right_elbow" />
         <limit lower="0.0" upper="${PI}" effort="${max_effort}" velocity="${max_velocity}"  />
@@ -116,4 +102,11 @@
       <axis xyz="0 1 0" />
       <parent link="${prefix}/${side}_wrist_0" />
+      <child link="${prefix}/${side}_wrist_1" />
+      <limit lower="${-PI_DIV_2}" upper="${PI_DIV_2}" effort="${max_effort}" velocity="${max_velocity}"  />
+    </joint>
+    <joint name="${side}_wrist_2" type="revolute">
+      <origin xyz="0 0 0" rpy="0 0 0" />
+      <axis xyz="1 0 0" />
+      <parent link="${prefix}/${side}_wrist_1" />
       <child link="${prefix}/${side}_wrist" />
       <limit lower="${-PI_DIV_2}" upper="${PI_DIV_2}" effort="${max_effort}" velocity="${max_velocity}"  />

File: urdf/xacro/human_leg.urdf.xacro (robot description, xacro)
@@ -61,5 +61,5 @@
         </joint>
     <!-- END hip -->
-    <joint name="${side}_knee" type="revolute">
+    <joint name="${side}_knee_0" type="revolute">
       <origin xyz="${thigh_length} 0 0" rpy="${PI_DIV_2} 0 0" />
       <axis xyz="0 0 1" />
