Commit message: update URDF

File: urdf/human.urdf (robot description, URDF)
Before this commit: robot human_model, 44 links, 43 joints
Links:
- link human/base: geometry visual cylinder length=-0.0763326765193 radius=0.123896225762
- link human/left_elbow: geometry visual cylinder length=0.270314394856 radius=0.025
- link human/left_hip: geometry visual cylinder length=0.559619800605 radius=0.05
- link human/left_knee: geometry visual cylinder length=0.352954406299 radius=0.025
- link human/left_shoulder: geometry visual cylinder length=0.298101187144 radius=0.05
- link human/neck: geometry visual cylinder length=0.181149056986 radius=0.04
- link human/right_elbow: geometry visual cylinder length=0.270314394856 radius=0.025
- link human/right_hip: geometry visual cylinder length=0.559619800605 radius=0.05
- link human/right_knee: geometry visual cylinder length=0.352954406299 radius=0.025
- link human/right_shoulder: geometry visual cylinder length=0.298101187144 radius=0.05
- link human/shoulder_center: geometry visual cylinder length=0.114356534425 radius=0.172633054012
- link human/spine: geometry visual cylinder length=0.260433842416 radius=0.152633054012
- link human/spine_0: geometry visual cylinder length=0.0868330314048 radius=0.132633054012
Joints:
- joint head: origin xyz=0 0 0.198713359681 rpy=0 0 0 -> xyz=0 0 0.181149056986 rpy=0 0 0
- joint left_ankle_0: origin xyz=0.36903984413 0 0 rpy=-1.57079632679 0 1.57079632679 -> xyz=0.352954406299 0 0 rpy=-1.57079632679 0 1.57079632679
- joint left_arm_mount: origin xyz=0 0.173623764208 -0.00143826424372 rpy=0 0 1.57079632679 -> xyz=0 0.172633054012 -0.00503493917921 rpy=0 0 1.57079632679
- joint left_elbow_0: origin xyz=0.343212242182 0 0 rpy=0 0 0 -> xyz=0.298101187144 0 0 rpy=0 0 0
- joint left_hip_leg_mount: origin xyz=0 0.0780638095132 -0.076637666482 rpy=0 1.57079632679 0 -> xyz=0 0.0738962257622 -0.0763326765193 rpy=0 1.57079632679 0
- joint left_knee_0: origin xyz=0.53151880807 0 0 rpy=1.57079632679 0 0 -> xyz=0.559619800605 0 0 rpy=1.57079632679 0 0
- joint left_wrist_0: origin xyz=0.273206361701 0 0 rpy=0 0 0 -> xyz=0.270314394856 0 0 rpy=0 0 0
- joint neck_0: origin xyz=0 0 0.126849441152 rpy=0 0 0 -> xyz=0 0 0.114356534425 rpy=0 0 0
- joint right_ankle_0: origin xyz=0.36903984413 0 0 rpy=-1.57079632679 0 1.57079632679 -> xyz=0.352954406299 0 0 rpy=-1.57079632679 0 1.57079632679
- joint right_arm_mount: origin xyz=0 -0.173623764208 -0.00143826424372 rpy=0 0 -1.57079632679 -> xyz=0 -0.172633054012 -0.00503493917921 rpy=0 0 -1.57079632679
- joint right_elbow_0: origin xyz=0.343212242182 0 0 rpy=0 0 0 -> xyz=0.298101187144 0 0 rpy=0 0 0
- joint right_hip_leg_mount: origin xyz=0 -0.0780638095132 -0.076637666482 rpy=0 1.57079632679 0 -> xyz=0 -0.0738962257622 -0.0763326765193 rpy=0 1.57079632679 0
- joint right_knee_0: origin xyz=0.53151880807 0 0 rpy=1.57079632679 0 0 -> xyz=0.559619800605 0 0 rpy=1.57079632679 0 0
- joint right_wrist_0: origin xyz=0.273206361701 0 0 rpy=0 0 0 -> xyz=0.270314394856 0 0 rpy=0 0 0
- joint shoulder_center: origin xyz=0 0 0.262448400938 rpy=0 0 0 -> xyz=0 0 0.260433842416 rpy=0 0 0
- joint spine_0: origin xyz=0 0 0.0900777328402 rpy=0 0 0 -> xyz=0 0 0.0868330314048 rpy=0 0 0

Commit message: updated model

File: urdf/human.urdf (robot description, URDF)
Before this commit: robot human_model, 44 links, 43 joints
Links:
- link human/base: geometry visual cylinder length=-0.0814017124054 radius=0.132917081552
- link human/left_elbow: geometry visual cylinder length=0.294319255902 radius=0.025
- link human/left_hip: geometry visual cylinder length=0.5886108303 radius=0.05
- link human/left_knee: geometry visual cylinder length=0.408774437278 radius=0.025
- link human/left_shoulder: geometry visual cylinder length=0.33692616474 radius=0.05
- link human/neck: geometry visual cylinder length=0.204191118591 radius=0.04
- link human/right_elbow: geometry visual cylinder length=0.294319255902 radius=0.025
- link human/right_hip: geometry visual cylinder length=0.5886108303 radius=0.05
- link human/right_knee: geometry visual cylinder length=0.408774437278 radius=0.025
- link human/right_shoulder: geometry visual cylinder length=0.33692616474 radius=0.05
- link human/shoulder_center: geometry visual cylinder length=0.121709143845 radius=0.184930241109
- link human/spine: geometry visual cylinder length=0.280112716739 radius=0.164930241109
- link human/spine_0: geometry visual cylinder length=0.0793042185134 radius=0.144930241109
Joints:
- joint head: origin xyz=0 0 0.181149056986 rpy=0 0 0 -> xyz=0 0 0.204191118591 rpy=0 0 0
- joint left_ankle_0: origin xyz=0.352954406299 0 0 rpy=-1.57079632679 0 1.57079632679 -> xyz=0.408774437278 0 0 rpy=-1.57079632679 0 1.57079632679
- joint left_arm_mount: origin xyz=0 0.172633054012 -0.00503493917921 rpy=0 0 1.57079632679 -> xyz=0 0.184930241109 0.00185424741055 rpy=0 0 1.57079632679
- joint left_elbow_0: origin xyz=0.298101187144 0 0 rpy=0 0 0 -> xyz=0.33692616474 0 0 rpy=0 0 0
- joint left_hip_leg_mount: origin xyz=0 0.0738962257622 -0.0763326765193 rpy=0 1.57079632679 0 -> xyz=0 0.082917081552 -0.0814017124054 rpy=0 1.57079632679 0
- joint left_knee_0: origin xyz=0.559619800605 0 0 rpy=1.57079632679 0 0 -> xyz=0.5886108303 0 0 rpy=1.57079632679 0 0
- joint left_wrist_0: origin xyz=0.270314394856 0 0 rpy=0 0 0 -> xyz=0.294319255902 0 0 rpy=0 0 0
- joint neck_0: origin xyz=0 0 0.114356534425 rpy=0 0 0 -> xyz=0 0 0.121709143845 rpy=0 0 0
- joint right_ankle_0: origin xyz=0.352954406299 0 0 rpy=-1.57079632679 0 1.57079632679 -> xyz=0.408774437278 0 0 rpy=-1.57079632679 0 1.57079632679
- joint right_arm_mount: origin xyz=0 -0.172633054012 -0.00503493917921 rpy=0 0 -1.57079632679 -> xyz=0 -0.184930241109 0.00185424741055 rpy=0 0 -1.57079632679
- joint right_elbow_0: origin xyz=0.298101187144 0 0 rpy=0 0 0 -> xyz=0.33692616474 0 0 rpy=0 0 0
- joint right_hip_leg_mount: origin xyz=0 -0.0738962257622 -0.0763326765193 rpy=0 1.57079632679 0 -> xyz=0 -0.082917081552 -0.0814017124054 rpy=0 1.57079632679 0
- joint right_knee_0: origin xyz=0.559619800605 0 0 rpy=1.57079632679 0 0 -> xyz=0.5886108303 0 0 rpy=1.57079632679 0 0
- joint right_wrist_0: origin xyz=0.270314394856 0 0 rpy=0 0 0 -> xyz=0.294319255902 0 0 rpy=0 0 0
- joint shoulder_center: origin xyz=0 0 0.260433842416 rpy=0 0 0 -> xyz=0 0 0.280112716739 rpy=0 0 0
- joint spine_0: origin xyz=0 0 0.0868330314048 rpy=0 0 0 -> xyz=0 0 0.0793042185134 rpy=0 0 0

Commit message: Code working at LASA

File: urdf/human.urdf (robot description, URDF)
Before this commit: robot human_model, 44 links, 43 joints
Links:
- link human/base: geometry visual cylinder length=-0.0811138121076 radius=0.130553532998
- link human/left_elbow: geometry visual cylinder length=0.274149473988 radius=0.025
- link human/left_hip: geometry visual cylinder length=0.564421893516 radius=0.05
- link human/left_knee: geometry visual cylinder length=0.407337097232 radius=0.025
- link human/left_shoulder: geometry visual cylinder length=0.294151609476 radius=0.05
- link human/neck: geometry visual cylinder length=0.204279422944 radius=0.04
- link human/right_elbow: geometry visual cylinder length=0.274149473988 radius=0.025
- link human/right_hip: geometry visual cylinder length=0.564421893516 radius=0.05
- link human/right_knee: geometry visual cylinder length=0.407337097232 radius=0.025
- link human/right_shoulder: geometry visual cylinder length=0.294151609476 radius=0.05
- link human/shoulder_center: geometry visual cylinder length=0.10127011497 radius=0.181172520845
- link human/spine: geometry visual cylinder length=0.275888061853 radius=0.161172520845
- link human/spine_0: geometry visual cylinder length=0.0726248956383 radius=0.141172520845
Joints:
- joint head: origin xyz=0 0 0.181149056986 rpy=0 0 0 -> xyz=0 0 0.204279422944 rpy=0 0 0
- joint left_ankle_0: origin xyz=0.352954406299 0 0 rpy=-1.57079632679 0 1.57079632679 -> xyz=0.407337097232 0 0 rpy=-1.57079632679 0 1.57079632679
- joint left_arm_mount: origin xyz=0 0.172633054012 -0.00503493917921 rpy=0 0 1.57079632679 -> xyz=0 0.181172520845 -0.00609526854636 rpy=0 0 1.57079632679
- joint left_elbow_0: origin xyz=0.298101187144 0 0 rpy=0 0 0 -> xyz=0.294151609476 0 0 rpy=0 0 0
- joint left_hip_leg_mount: origin xyz=0 0.0738962257622 -0.0763326765193 rpy=0 1.57079632679 0 -> xyz=0 0.080553532998 -0.0811138121076 rpy=0 1.57079632679 0
- joint left_knee_0: origin xyz=0.559619800605 0 0 rpy=1.57079632679 0 0 -> xyz=0.564421893516 0 0 rpy=1.57079632679 0 0
- joint left_wrist_0: origin xyz=0.270314394856 0 0 rpy=0 0 0 -> xyz=0.274149473988 0 0 rpy=0 0 0
- joint neck_0: origin xyz=0 0 0.114356534425 rpy=0 0 0 -> xyz=0 0 0.10127011497 rpy=0 0 0
- joint right_ankle_0: origin xyz=0.352954406299 0 0 rpy=-1.57079632679 0 1.57079632679 -> xyz=0.407337097232 0 0 rpy=-1.57079632679 0 1.57079632679
- joint right_arm_mount: origin xyz=0 -0.172633054012 -0.00503493917921 rpy=0 0 -1.57079632679 -> xyz=0 -0.181172520845 -0.00609526854636 rpy=0 0 -1.57079632679
- joint right_elbow_0: origin xyz=0.298101187144 0 0 rpy=0 0 0 -> xyz=0.294151609476 0 0 rpy=0 0 0
- joint right_hip_leg_mount: origin xyz=0 -0.0738962257622 -0.0763326765193 rpy=0 1.57079632679 0 -> xyz=0 -0.080553532998 -0.0811138121076 rpy=0 1.57079632679 0
- joint right_knee_0: origin xyz=0.559619800605 0 0 rpy=1.57079632679 0 0 -> xyz=0.564421893516 0 0 rpy=1.57079632679 0 0
- joint right_wrist_0: origin xyz=0.270314394856 0 0 rpy=0 0 0 -> xyz=0.274149473988 0 0 rpy=0 0 0
- joint shoulder_center: origin xyz=0 0 0.260433842416 rpy=0 0 0 -> xyz=0 0 0.275888061853 rpy=0 0 0
- joint spine_0: origin xyz=0 0 0.0868330314048 rpy=0 0 0 -> xyz=0 0 0.0726248956383 rpy=0 0 0
